File: pcb/main/pHMeter.kicad_pcb (KiCad board)
At the start: 2 copper layers, 100 x 87 mm, 148 parts, among them J1 Conn_02x03_Odd_Even, J2 Conn_Coaxial_Power, J3 Conn_Coaxial_Power, J4 AudioJack3_SwitchTR, J5 RJ12, J6 AudioJack3_SwitchTR, J7 SJ, J8 SJ, Q1 ZXMS6004, Q2 ZXMS6004, Q3 DMP1045, Q4 ZXMS6004, Q5 ZXMS6004, SW1 Rotary_Encoder_Switch, U1 TLV6004PW, U2 TLV6004PW, U3 ATMEGA32U4-AU, U4 MCP1703A, U5 AP63203WU-7, U6 HX711, U7 SST26VF064B, U9 MCP73811T, X1 MINI-USB-SCHIELD-32005-201, Y1 Crystal

Commit message: update pcb
Parts:
- JP3, JP4, JP6, JP7: footprint Connector_PinHeader_2.54mm:PinHeader_1x02_P2.54mm_Vertical -> Connector_Molex:Molex_KK-254_AE-6410-02A_1x02_P2.54mm_Vertical
- RV1: footprint Potentiometer_THT:Potentiometer_Bourns_3339P_Vertical_HandSoldering -> Potentiometer_THT:Potentiometer_Bourns_3339S_Horizontal
- moved R26 195.0 mm to (227.1, 72.6), turned to 180 degrees
- moved R27 193.7 mm to (227.1, 85.1), turned to 180 degrees
- moved D13 191.2 mm to (221.0, 72.6)
- moved D12 189.9 mm to (221.0, 85.1)
- moved Q1 189.3 mm to (227.3, 80.2), turned to 270 degrees
- moved Q2 188.2 mm to (227.3, 92.7), turned to 270 degrees
- moved JP4 178.5 mm to (220.0, 78.7)
- moved JP3 177.1 mm to (220.0, 91.2)
- moved JP1 154.8 mm to (225.8, 108.0)
- moved JP2 154.8 mm to (225.8, 113.5)
- moved D4 154.4 mm to (273.9, 128.3), turned to 0 degrees
- moved C22 154.4 mm to (245.4, 105.9), turned to 180 degrees
- moved D9 153.3 mm to (252.0, 94.0), turned to 180 degrees
- moved C6 152.5 mm to (274.4, 125.7), turned to 0 degrees
- moved D10 150.6 mm to (252.0, 97.5), turned to 180 degrees
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Connections:
- DS1 pad 11: D9 -> D8
- DS1 pad 12: D11 -> D9
- DS1 pad 13: D5 -> D10
- DS1 pad 14: D10 -> D5
- Q1 pad 1: D8 -> D11
- Q4 pad 1: D12 -> A2
- Q5 pad 1: D12 -> A3
- R26 pad 1: D8 -> D11
- R47 pad 1: D12 -> A2
- R48 pad 1: D12 -> A3
- SW1 pad A: Net-(SW1-PadA) -> TX
- SW1 pad B: Net-(SW1-PadB) -> RX
- SW1 pad S1: Net-(SW1-PadS1) -> D11
- SW1 pad S2: Net-(SW1-PadS2) -> GND
Other:
- board text added: "1"
- board text added: "2"
- board text added: "3"
- board text added: "4"
- board text added: "ADC"
- board text added: "I/O"
- board text added: "RX"
- board text added: "TX"
- board text removed: "Foods"

Commit message: Created making doc and PCB for revision
Parts:
- JP5: footprint Connector_PinHeader_2.54mm:PinHeader_1x02_P2.54mm_Vertical -> Connector_Molex:Molex_KK-254_AE-6410-02A_1x02_P2.54mm_Vertical
- RV1: moved to B.Cu
- moved RV1 5.08 mm to (273.6, 106.9)
- moved D4 4.30 mm to (269.6, 128.1), turned to 180 degrees
- moved R32 3.81 mm to (272.8, 111.8)
- moved R33 3.30 mm to (276.4, 111.8)
- moved C22 3.06 mm to (245.6, 102.9)
- moved D15 3.06 mm to (248.7, 115.8)
- moved R39 3.06 mm to (249.9, 112.3)
- moved U5 3.06 mm to (246.1, 107.5)
- moved C19 3.06 mm to (246.6, 112.3)
- moved C24 3.06 mm to (243.1, 112.3)
- moved C25 3.06 mm to (239.5, 112.3)
- moved D16 3.06 mm to (237.2, 115.8)
- moved R40 3.06 mm to (236.1, 112.3)
- moved L2 3.06 mm to (239.3, 105.9)
- moved D14 3.05 mm to (246.4, 129.5)
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Connections:
- C33 pad 1: A3 -> A4
- R38 pad 2: A3 -> A4
- R45 pad 1: A3 -> A4
- SW1 pad S1: D11 -> D7
- U6 pad 11: D7 -> A1
- U6 pad 12: A5 -> A0
Routing:
- net 3.3V: track 0.00 -> 356.9 mm, vias 0 -> 10
- net 12V: track 0.00 -> 192.7 mm, vias 0 -> 2
- net D13: track 0.00 -> 137.1 mm, vias 0 -> 1
- net SDA: track 0.00 -> 116.2 mm, vias 0 -> 1
- net RX: track 0.00 -> 114.0 mm, vias 0 -> 1
- net SCL: track 0.00 -> 108.9 mm, vias 0 -> 1
- net D7: track 0.00 -> 86.9 mm
- net A4: track 0.00 -> 71.3 mm, vias 0 -> 2
- net VUSB: track 0.00 -> 68.1 mm, vias 0 -> 2
- net A5: track 0.00 -> 62.0 mm, vias 0 -> 4
- net USB_P: track 0.00 -> 59.3 mm, vias 0 -> 2
- net USB_N: track 0.00 -> 57.4 mm, vias 0 -> 2
- net VDD: track 0.00 -> 54.5 mm
- net Net-(DS1-Pad3): track 0.00 -> 53.3 mm
- net D11: track 0.00 -> 48.6 mm, vias 0 -> 2
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- added copper zone on B.Cu, net GND
- added copper zone on F.Cu, net GND
Other:
- board text added: "BAT"

Commit message: Update 3D for Rotary & BNC
Parts:
- moved SW1 11.9 mm to (191.0, 142.0), turned to 0 degrees
- moved J2 2.54 mm to (186.7, 124.2)
Routing:
- net RX: track 114.0 -> 120.4 mm
- net Net-(J2-Pad1): track 27.7 -> 28.8 mm
Changed lines of the file:
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@@
     (thickness 1.6)
     (drawings 75)
-    (tracks 991)
+    (tracks 994)
     (zones 0)
     (modules 148)
@@
   )
   (module Connector_Coaxial:BNC_TEConnectivity_1478204_Vertical (layer F.Cu)
-    (at 186.69 121.666)
+    (at 186.69 124.206)
     (descr "BNC female PCB mount 4 pin straight chassis connector http://www.te.com/usa-en/product-1-1478204-0.html")
     (tags "BNC female PCB mount 4 pin straight chassis connector ")
@@
       (rotate (xyz 0 0 0))
     )
+    (model ${KIPRJMOD}/3dmodels/bnc_with_plastic.stp
+      (at (xyz 0 0 0))
+      (scale (xyz 1.05 1 1.05))
+      (rotate (xyz -90 0 45))
+    )
   )
   (module Connector_Coaxial:BNC_TEConnectivity_1478204_Vertical (layer F.Cu)
@@
       (rotate (xyz 0 0 0))
     )
+    (model ${KIPRJMOD}/3dmodels/bnc_with_plastic.stp
+      (at (xyz 0 0 0))
+      (scale (xyz 1.05 1 1.05))
+      (rotate (xyz -90 0 45))
+    )
   )
   (module Jumper:SolderJumper-2_P1.3mm_Open_RoundedPad1.0x1.5mm (layer F.Cu)
@@
   )
   (module Rotary_Encoder:RotaryEncoder_Alps_EC11E-Switch_Vertical_H20mm (layer B.Cu)
-    (at 194.31 130.556 270)
+    (at 191.008 141.986)
     (descr "Alps rotary encoder, EC12E... with switch, vertical shaft, http://www.alps.com/prod/info/E/HTML/Encoder/Incremental/EC11/EC11E15204A3.html")
     (tags "rotary encoder")
-    (fp_text reference SW1 (at 2.8 4.7 270) (layer B.SilkS)
+    (fp_text reference SW1 (at 2.8 4.7 180) (layer B.SilkS)
       (effects (font (size 1 1) (thickness 0.15)) (justify mirror))
     )
-    (fp_text value Rotary_Encoder_Switch (at 7.5 -10.4 270) (layer B.Fab)
+    (fp_text value Rotary_Encoder_Switch (at 7.5 -10.4 180) (layer B.Fab)
       (effects (font (size 1 1) (thickness 0.15)) (justify mirror))
     )
@@
     (fp_line (start 7.5 -2) (end 7.5 -3) (layer B.SilkS) (width 0.12))
     (fp_line (start 7 -2.5) (end 8 -2.5) (layer B.SilkS) (width 0.12))
-    (fp_text user %R (at 11.1 -6.3 270) (layer B.Fab)
+    (fp_text user %R (at 11.1 -6.3 180) (layer B.Fab)
       (effects (font (size 1 1) (thickness 0.15)) (justify mirror))
     )
-    (pad S1 thru_hole circle (at 14.5 -5 270) (size 2 2) (drill 1) (layers *.Cu *.Mask)
+    (pad S1 thru_hole circle (at 14.5 -5) (size 2 2) (drill 1) (layers *.Cu *.Mask)
       (net 71 D7))
-    (pad S2 thru_hole circle (at 14.5 0 270) (size 2 2) (drill 1) (layers *.Cu *.Mask)
+    (pad S2 thru_hole circle (at 14.5 0) (size 2 2) (drill 1) (layers *.Cu *.Mask)
       (net 2 GND))
-    (pad MP thru_hole rect (at 7.5 -8.1 270) (size 3.2 2) (drill oval 2.8 1.5) (layers *.Cu *.Mask))
-    (pad MP thru_hole rect (at 7.5 3.1 270) (size 3.2 2) (drill oval 2.8 1.5) (layers *.Cu *.Mask))
-    (pad B thru_hole circle (at 0 -5 270) (size 2 2) (drill 1) (layers *.Cu *.Mask)
+    (pad MP thru_hole rect (at 7.5 -8.1) (size 3.2 2) (drill oval 2.8 1.5) (layers *.Cu *.Mask))
+    (pad MP thru_hole rect (at 7.5 3.1) (size 3.2 2) (drill oval 2.8 1.5) (layers *.Cu *.Mask))
+    (pad B thru_hole circle (at 0 -5) (size 2 2) (drill 1) (layers *.Cu *.Mask)
       (net 73 RX))
-    (pad C thru_hole circle (at 0 -2.5 270) (size 2 2) (drill 1) (layers *.Cu *.Mask)
+    (pad C thru_hole circle (at 0 -2.5) (size 2 2) (drill 1) (layers *.Cu *.Mask)
       (net 2 GND))
-    (pad A thru_hole rect (at 0 0 270) (size 2 2) (drill 1) (layers *.Cu *.Mask)
+    (pad A thru_hole rect (at 0 0) (size 2 2) (drill 1) (layers *.Cu *.Mask)
       (net 74 TX))
     (model ${KISYS3DMOD}/Rotary_Encoder.3dshapes/RotaryEncoder_Alps_EC11E-Switch_Vertical_H20mm.wrl
@@
       (rotate (xyz 0 0 0))
     )
+    (model ${KIPRJMOD}/3dmodels/AB2_ROT_ENC_W_SW.wrl
+      (offset (xyz 7.45 -2.5 0))
+      (scale (xyz 0.015 0.0153 0.015))
+      (rotate (xyz 0 0 -90))
+    )
   )
   (module Capacitor_SMD:C_0805_2012Metric_Pad1.15x1.40mm_HandSolder (layer F.Cu)
@@
   (gr_line (start 279.4 61.5696) (end 279.4 148.59) (layer Edge.Cuts) (width 0.05))
   (gr_line (start 179.4 61.5696) (end 279.4 61.5696) (layer Edge.Cuts) (width 0.05))
-  (via (at 252.8824 80.3148) (size 0.8) (drill 0.4) (layers F.Cu B.Cu) (net 2))
-  (via (at 256.1082 83.7438) (size 0.8) (drill 0.4) (layers F.Cu B.Cu) (net 2))
   (via (at 268.732 89.1794) (size 0.8) (drill 0.4) (layers F.Cu B.Cu) (net 1))
   (via (at 268.732 86.106) (size 0.8) (drill 0.4) (layers F.Cu B.Cu) (net 1))
@@
   (via (at 216.5768 97.4688) (size 0.8) (drill 0.4) (layers F.Cu B.Cu) (net 1))
   (segment (start 213.8463 94.7383) (end 216.5768 97.4688) (width 0.25) (layer B.Cu) (net 1))
+  (via (at 252.8824 80.3148) (size 0.8) (drill 0.4) (layers F.Cu B.Cu) (net 2))
+  (via (at 256.1082 83.7438) (size 0.8) (drill 0.4) (layers F.Cu B.Cu) (net 2))
   (segment (start 257.066 123.444) (end 257.048 123.462) (width 0.508) (layer F.Cu) (net 2))
   (via (at 264.1346 119.6594) (size 0.8) (drill 0.4) (layers F.Cu B.Cu) (net 2))
@@
   (segment (start 204.234 108.901942) (end 203.058058 107.726) (width 0.25) (layer F.Cu) (net 46))
   (segment (start 204.234 110.49) (end 204.234 108.901942) (width 0.25) (layer F.Cu) (net 46))
-  (segment (start 195.834 121.666) (end 186.69 121.666) (width 0.25) (layer F.Cu) (net 46))
   (segment (start 203.24649 111.47751) (end 203.24649 114.25351) (width 0.25) (layer F.Cu) (net 46))
   (segment (start 203.24649 114.25351) (end 195.834 121.666) (width 0.25) (layer F.Cu) (net 46))
   (segment (start 204.234 110.49) (end 203.24649 111.47751) (width 0.25) (layer F.Cu) (net 46))
+  (segment (start 193.294 124.206) (end 195.834 121.666) (width 0.25) (layer F.Cu) (net 46))
+  (segment (start 186.69 124.206) (end 193.294 124.206) (width 0.25) (layer F.Cu) (net 46))
   (segment (start 183.515 110.617) (end 189.865 110.617) (width 0.25) (layer F.Cu) (net 47))
   (segment (start 189.865 110.617) (end 189.865 104.267) (width 0.25) (layer F.Cu) (net 47))
@@
   (segment (start 241.559397 76.236999) (end 243.300398 77.978) (width 0.25) (layer B.Cu) (net 73))
   (segment (start 217.895001 76.236999) (end 241.559397 76.236999) (width 0.25) (layer B.Cu) (net 73))
-  (segment (start 199.31 130.556) (end 195.16699 126.41299) (width 0.25) (layer B.Cu) (net 73))
   (segment (start 195.16699 98.96501) (end 217.895001 76.236999) (width 0.25) (layer B.Cu) (net 73))
   (segment (start 195.16699 126.41299) (end 195.16699 98.96501) (width 0.25) (layer B.Cu) (net 73))
@@
   (segment (start 260.998 77.102) (end 260.858 76.962) (width 0.25) (layer F.Cu) (net 73))
   (segment (start 262.748 77.102) (end 260.998 77.102) (width 0.25) (layer F.Cu) (net 73))
+  (segment (start 195.16699 126.41299) (end 195.16699 129.95301) (width 0.25) (layer B.Cu) (net 73))
+  (segment (start 191.008 134.112) (end 191.008 136.986) (width 0.25) (layer B.Cu) (net 73))
+  (segment (start 195.16699 129.95301) (end 191.008 134.112) (width 0.25) (layer B.Cu) (net 73))
   (segment (start 255.524 107.442) (end 255.524 105.156) (width 0.25) (layer F.Cu) (net 74))
   (segment (start 261.931991 90.053597) (end 264.384794 87.600794) (width 0.25) (layer F.Cu) (net 74))

Commit message: Update PCB connection, run ERC and update pinMapping.md
Routing:
- net TX: track 41.3 -> 184.9 mm, vias 2 -> 4
- net D7: track 86.9 -> 117.3 mm
- net VBAT: track 9.94 -> 36.1 mm, vias 0 -> 2
- net GND: track 35.4 -> 42.4 mm, vias 16 -> 17
- net Net-(D10-Pad2): track 0.00 -> 3.04 mm
- net 3.3V: track 356.9 -> 357.5 mm
