File: pcb/main/pHMeter.kicad_pcb (KiCad board)
At the start: 2 copper layers, 100 x 87 mm, 148 parts, among them J1 Conn_02x03_Odd_Even, J2 Conn_Coaxial_Power, J3 Conn_Coaxial_Power, J4 AudioJack3_SwitchTR, J5 RJ12, J6 AudioJack3_SwitchTR, J7 SJ, J8 SJ, Q1 ZXMS6004, Q2 ZXMS6004, Q3 DMP1045, Q4 ZXMS6004, Q5 ZXMS6004, SW1 Rotary_Encoder_Switch, U1 TLV6004PW, U2 TLV6004PW, U3 ATMEGA32U4-AU, U4 MCP1703A, U5 AP63203WU-7, U6 HX711, U7 SST26VF064B, U9 MCP73811T, X1 MINI-USB-SCHIELD-32005-201, Y1 Crystal

Commit message: Replace minimum track 8mil -> 16 mil
Parts:
- moved R20 5.40 mm to (246.9, 73.7), turned to 270 degrees
- moved D8 3.41 mm to (244.9, 73.7), turned to 270 degrees
- moved R36 0.75 mm to (248.9, 73.7), turned to 90 degrees
- moved C11 0.25 mm to (258.6, 88.6)
- moved R6 0.24 mm to (204.2, 99.3)
Routing:
- net GND: track 42.4 -> 48.0 mm, vias 17 -> 18
- net D13: track 137.1 -> 141.0 mm
- net 3.3V: track 357.5 -> 355.9 mm, vias 10 -> 12
- net SDA: track 116.2 -> 117.6 mm
- net /24bits ADC/LGND: track 18.6 -> 19.9 mm
- net Net-(C2-Pad2): track 23.5 -> 24.6 mm
- net D11: track 48.6 -> 49.6 mm
- net Net-(C3-Pad1): track 11.3 -> 12.3 mm
- net MOSI: track 44.0 -> 43.1 mm
- net D5: track 33.0 -> 32.1 mm
- net MISO: track 39.2 -> 38.4 mm
- net USB_N: track 57.4 -> 58.1 mm
- net HWB: track 3.91 -> 4.61 mm
- net A+: track 30.5 -> 31.2 mm
- net A4: track 71.3 -> 71.9 mm
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Other:
- net class Default: trace_width 0.25 -> 0.4064
- net class Luc added: clearance 0.2, trace_width 0.4064, via_dia 0.8, via_drill 0.4
- rule trace_min: 0.2 -> 0.406

Commit message: chore: add label v0.1 on pcb
Other:
- board text added: "pHMeter v0.1"

Commit message: Fix MOSFET ZXMS6004 pin mapping
Connections:
- Q1 pad 2: Net-(JP4-Pad2) -> GND
- Q1 pad 3: GND -> Net-(JP4-Pad2)
- Q2 pad 2: Net-(JP3-Pad2) -> GND
- Q2 pad 3: GND -> Net-(JP3-Pad2)
- Q4 pad 2: Net-(JP6-Pad2) -> GND
- Q4 pad 3: GND -> Net-(JP6-Pad2)
- Q5 pad 2: Net-(JP7-Pad2) -> GND
- Q5 pad 3: GND -> Net-(JP7-Pad2)
Routing:
- net Net-(JP3-Pad2): track 4.09 -> 5.86 mm
- net Net-(JP7-Pad2): track 3.85 -> 5.62 mm
- net Net-(JP6-Pad2): track 3.85 -> 5.62 mm
- net Net-(JP4-Pad2): track 4.02 -> 5.80 mm
