File: pcb/main/pHMeter.kicad_pcb (KiCad board)
At the start: 2 copper layers, 100 x 87 mm, 148 parts, among them J1 Conn_02x03_Odd_Even, J2 Conn_Coaxial_Power, J3 Conn_Coaxial_Power, J4 AudioJack3_SwitchTR, J5 RJ12, J6 AudioJack3_SwitchTR, J7 SJ, J8 SJ, Q1 ZXMS6004, Q2 ZXMS6004, Q3 DMP1045, Q4 ZXMS6004, Q5 ZXMS6004, SW1 Rotary_Encoder_Switch, U1 TLV6004PW, U2 TLV6004PW, U3 ATMEGA32U4-AU, U4 MCP1703A, U5 AP63203WU-7, U6 HX711, U7 SST26VF064B, U9 MCP73811T, X1 MINI-USB-SCHIELD-32005-201, Y1 Crystal

Commit message: Fix: Changed inductor size (issue #4)
Parts:
- C13, C14: value 22pF -> 18pF
- C18: value 100nF -> 1uF
- L2: footprint Inductor_SMD:L_TDK_SLF6028 -> Inductor_SMD:L_Taiyo-Yuden_NR-40xx_HandSoldering
- R20, R21, R23, R24: value 10k -> 1k

Commit message: Fix: renamed value for LEDs
Parts:
- C13, C14: value 18pF -> 18p
- C15, C16, C17, C26, C28, C30: value 100nF -> 100n
- C18: value 1uF -> 1u
- C27, C29: value 10uF -> 10u
- D1, D2: value D -> D_Schottky
- RV1: footprint Potentiometer_THT:Potentiometer_Bourns_3339S_Horizontal -> Potentiometer_THT:Potentiometer_Bourns_3339P_Vertical_HandSoldering
- moved RV1 5.34 mm to (273.7, 101.6)
Connections:
- RV1 pad 1: Net-(R32-Pad2) -> Net-(R33-Pad1)
- RV1 pad 3: Net-(R33-Pad1) -> Net-(R32-Pad2)

Commit message: Updated: New version for board
Parts:
- removed C30: 100n, Capacitor_SMD:C_0805_2012Metric_Pad1.15x1.40mm_HandSolder
- D1, D14, D2, D3, D4, D5: value D_Schottky -> MBR0520LT1G
- D10, D11, D9: value LED -> YELLOW
- D12, D13, D17, D18: value LED -> BLUE
- D15, D16: value RED -> GREEN
- D19, D20: value TX -> YELLOW
- D7, D8: value LED -> GREEN
- moved SJ1 1.53 mm to (213.4, 86.4), turned to 180 degrees
Routing:
- net Net-(U6-Pad6): track 3.63 -> 0.00 mm
- net /24bits ADC/LGND: track 19.9 -> 18.4 mm
- net Net-(C2-Pad2): track 24.6 -> 25.9 mm

Commit message: fix: refactor hardware design
Parts:
- moved D4 129.9 mm to (140.3, 116.5)
- moved C1 129.9 mm to (63.3, 72.3)
- moved C10 129.9 mm to (68.5, 93.9)
- moved C11 129.9 mm to (129.2, 77.1)
- moved C18 129.9 mm to (127.2, 76.9)
- moved C21 129.9 mm to (127.7, 110.9)
- moved C22 129.9 mm to (116.2, 91.4)
- moved C23 129.9 mm to (129.9, 115.0)
- moved C24 129.9 mm to (113.7, 100.7)
- moved C26 129.9 mm to (75.1, 74.6)
- moved C28 129.9 mm to (79.4, 73.6)
- moved C29 129.9 mm to (79.4, 77.1)
- moved C3 129.9 mm to (63.3, 74.6)
- moved C31 129.9 mm to (136.6, 93.6)
- moved C33 129.9 mm to (123.1, 118.3)
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