File: pcb/main/pH.sch (KiCad schematic (older format))
At the start: 9 parts, among them J3 Conn_Coaxial_Power, U1 TLV6004PW

Commit message: Fix: renamed value for LEDs
Parts:
- C1, C3: Description (none) -> Multilayer Ceramic Capacitors MLCC - SMD/SMT WCAP-CSGP 0.1u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; MFN (none) -> Wurth Elektronik; MFP (none) -> 885012207072; S1PL (none) -> https://www.mouser.com/ProductDetail/Wurth-Elektronik/88501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; S1PN (none) -> 710-885012207072
- C9: Description (none) -> Multilayer Ceramic Capacitors MLCC - SMD/SMT 6.3V 22uF X5R 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; MFN (none) -> Samsung Electro-Mechanics; MFP (none) -> CL21A226KQCLRNC; S1PL (none) -> https://www.mouser.com/ProductDetail/Samsung-Electro-Mechan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; S1PN (none) -> 187-CL21A226KQCLRNC
Changed lines of the file:
@@
 F 1 "100n" H 4665 4455 50  0000 L CNN
 F 2 "Capacitor_SMD:C_0805_2012Metric_Pad1.15x1.40mm_HandSolder" H 4588 4350 50  0001 C CNN
-F 3 "~" H 4550 4500 50  0001 C CNN
+F 3 "https://www.mouser.com/datasheet/2/445/885012207072-1727745.pdf" H 4550 4500 50  0001 C CNN
+F 4 "Multilayer Ceramic Capacitors MLCC - SMD/SMT WCAP-CSGP 0.1uF 0805 10% 25V MLCC " H 4550 4500 50  0001 C CNN "Description"
+F 5 "Wurth Elektronik " H 4550 4500 50  0001 C CNN "MFN"
+F 6 "885012207072" H 4550 4500 50  0001 C CNN "MFP"
+F 7 "https://www.mouser.com/ProductDetail/Wurth-Elektronik/885012207072?qs=0KOYDY2FL28rQMV4504TxA%3D%3D" H 4550 4500 50  0001 C CNN "S1PL"
+F 8 "710-885012207072 " H 4550 4500 50  0001 C CNN "S1PN"
 	1    4550 4500
 	1    0    0    -1
@@
 F 1 "22u" H 7915 4355 50  0000 L CNN
 F 2 "Capacitor_SMD:C_0805_2012Metric_Pad1.15x1.40mm_HandSolder" H 7838 4250 50  0001 C CNN
-F 3 "~" H 7800 4400 50  0001 C CNN
+F 3 "https://www.mouser.com/datasheet/2/585/MLCC-1837944.pdf" H 7800 4400 50  0001 C CNN
+F 4 "Multilayer Ceramic Capacitors MLCC - SMD/SMT 6.3V 22uF X5R 10% 0805" H 7800 4400 50  0001 C CNN "Description"
+F 5 "Samsung Electro-Mechanics " H 7800 4400 50  0001 C CNN "MFN"
+F 6 "CL21A226KQCLRNC" H 7800 4400 50  0001 C CNN "MFP"
+F 7 "https://www.mouser.com/ProductDetail/Samsung-Electro-Mechanics/CL21A226KQCLRNC?qs=xZ%2FP%252Ba9zWqYG0ePGTF%2FymQ%3D%3D" H 7800 4400 50  0001 C CNN "S1PL"
+F 8 " 187-CL21A226KQCLRNC " H 7800 4400 50  0001 C CNN "S1PN"
 	1    7800 4400
 	1    0    0    -1
@@
 F 1 "100n" H 3965 4055 50  0000 L CNN
 F 2 "Capacitor_SMD:C_0805_2012Metric_Pad1.15x1.40mm_HandSolder" H 3888 3950 50  0001 C CNN
-F 3 "~" H 3850 4100 50  0001 C CNN
+F 3 "https://www.mouser.com/datasheet/2/445/885012207072-1727745.pdf" H 3850 4100 50  0001 C CNN
+F 4 "Multilayer Ceramic Capacitors MLCC - SMD/SMT WCAP-CSGP 0.1uF 0805 10% 25V MLCC " H 3850 4100 50  0001 C CNN "Description"
+F 5 "Wurth Elektronik " H 3850 4100 50  0001 C CNN "MFN"
+F 6 "885012207072" H 3850 4100 50  0001 C CNN "MFP"
+F 7 "https://www.mouser.com/ProductDetail/Wurth-Elektronik/885012207072?qs=0KOYDY2FL28rQMV4504TxA%3D%3D" H 3850 4100 50  0001 C CNN "S1PL"
+F 8 "710-885012207072 " H 3850 4100 50  0001 C CNN "S1PN"
 	1    3850 4100
 	1    0    0    -1

Commit message: Fix: Changed BNC connector for pH and conductometer (issue #3)
Parts:
- J3: Description (none) -> RF Connectors / Coaxial Connectors BNC ST PCB JACK 50 OHM T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; MFN (none) -> Amphenol RF; MFP (none) -> 112404; S1PL (none) -> https://www.mouser.com/ProductDetail/Amphenol-RF/112404?qs=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; S1PN (none) -> 523-112404
Changed lines of the file:
@@
 F 1 "Conn_Coaxial_Power" V 6124 4000 50  0000 C CNN
 F 2 "Connector_Coaxial:BNC_TEConnectivity_1478204_Vertical" H 6250 4000 50  0001 C CNN
-F 3 "~" H 6250 4000 50  0001 C CNN
+F 3 "https://www.mouser.com/datasheet/2/18/112404-714699.pdf" H 6250 4000 50  0001 C CNN
+F 4 "RF Connectors / Coaxial Connectors BNC ST PCB JACK 50 OHM TF-4 POST " H 6250 4050 50  0001 C CNN "Description"
+F 5 "Amphenol RF " H 6250 4050 50  0001 C CNN "MFN"
+F 6 "112404 " H 6250 4050 50  0001 C CNN "MFP"
+F 7 "https://www.mouser.com/ProductDetail/Amphenol-RF/112404?qs=sGAEpiMZZMvlX3nhDDO4ALoCC5VwNXaExnhG12ncsBA=" H 6250 4050 50  0001 C CNN "S1PL"
+F 8 "523-112404" H 6250 4050 50  0001 C CNN "S1PN"
 	1    6250 4050
 	0    1    1    0
