File: pcb/main/pHMeter.sch (KiCad schematic (older format))
At the start: 90 parts, among them J1 Conn_02x03_Odd_Even, J4 AudioJack3_SwitchTR, J5 RJ12, J6 AudioJack3_SwitchTR, J7 SJ, Q1 ZXMS6004, Q2 ZXMS6004, Q3 DMP1045, Q4 ZXMS6004, Q5 ZXMS6004, SW1 Rotary_Encoder_Switch, U3 ATMEGA32U4-AU, U4 MCP1703A, U9 MCP73811T, X1 MINI-USB-SCHIELD-32005-201, Y1 Crystal

Commit message: Fix: Changed BNC connector for pH and conductometer (issue #3)
Parts:
- D10, D11, D19, D20, D9: Description (none) -> Standard LEDs - SMD WL-SMCW SMDMono TpVw Waterclr 0805 Yell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; MFN (none) -> Wurth Elektronik; MFP (none) -> 150080YS75000; S1PL (none) -> https://www.mouser.com/ProductDetail/Wurth-Elektronik/15008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; S1PN (none) -> 710-150080YS75000
- D12, D13, D17, D18: Description (none) -> Standard LEDs - SMD WL-SMCW SMDMono TpVw Waterclr 0805 Blue; MFN (none) -> Wurth Elektronik; MFP (none) -> 150080BS75000; S1PL (none) -> https://www.mouser.com/ProductDetail/Wurth-Elektronik/15008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; S1PN (none) -> 710-150080BS75000
- D7, D8: Description (none) -> Standard LEDs - SMD WL-SMCW SMDMono TpVw Waterclr 0805 Green; MFN (none) -> Wurth Elektronik; MFP (none) -> 150080GS75000; S1PL (none) -> https://www.mouser.com/ProductDetail/Wurth-Elektronik/15008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; S1PN (none) -> 710-150080GS75000
Changed lines of the file:
@@
 F 1 "BLUE" H 9018 3601 50  0000 C CNN
 F 2 "LED_SMD:LED_0805_2012Metric_Pad1.15x1.40mm_HandSolder" H 9025 3475 50  0001 C CNN
-F 3 "~" H 9025 3475 50  0001 C CNN
+F 3 "https://www.mouser.com/datasheet/2/445/150080BS75000-1715853.pdf" H 9025 3475 50  0001 C CNN
+F 4 "Standard LEDs - SMD WL-SMCW SMDMono TpVw Waterclr 0805 Blue " H 9025 3475 50  0001 C CNN "Description"
+F 5 "Wurth Elektronik " H 9025 3475 50  0001 C CNN "MFN"
+F 6 "150080BS75000 " H 9025 3475 50  0001 C CNN "MFP"
+F 7 "https://www.mouser.com/ProductDetail/Wurth-Elektronik/150080BS75000?qs=2kOmHSv6VfT2tBo3UPVqAQ%3D%3D" H 9025 3475 50  0001 C CNN "S1PL"
+F 8 " 710-150080BS75000 " H 9025 3475 50  0001 C CNN "S1PN"
 	1    9025 3475
 	-1   0    0    -1
@@
 F 1 "BLUE" H 9018 2026 50  0000 C CNN
 F 2 "LED_SMD:LED_0805_2012Metric_Pad1.15x1.40mm_HandSolder" H 9025 1900 50  0001 C CNN
-F 3 "~" H 9025 1900 50  0001 C CNN
+F 3 "https://www.mouser.com/datasheet/2/445/150080BS75000-1715853.pdf" H 9025 1900 50  0001 C CNN
+F 4 "Standard LEDs - SMD WL-SMCW SMDMono TpVw Waterclr 0805 Blue " H 9025 1900 50  0001 C CNN "Description"
+F 5 "Wurth Elektronik " H 9025 1900 50  0001 C CNN "MFN"
+F 6 "150080BS75000 " H 9025 1900 50  0001 C CNN "MFP"
+F 7 "https://www.mouser.com/ProductDetail/Wurth-Elektronik/150080BS75000?qs=2kOmHSv6VfT2tBo3UPVqAQ%3D%3D" H 9025 1900 50  0001 C CNN "S1PL"
+F 8 " 710-150080BS75000 " H 9025 1900 50  0001 C CNN "S1PN"
 	1    9025 1900
 	-1   0    0    -1
@@
 F 1 "GREEN" V 6423 4330 50  0000 L CNN
 F 2 "LED_SMD:LED_0805_2012Metric_Pad1.15x1.40mm_HandSolder" H 6475 4250 50  0001 C CNN
-F 3 "~" H 6475 4250 50  0001 C CNN
+F 3 "https://www.mouser.com/datasheet/2/445/150080GS75000-1715657.pdf" H 6475 4250 50  0001 C CNN
+F 4 "Standard LEDs - SMD WL-SMCW SMDMono TpVw Waterclr 0805 Green " H 6475 4250 50  0001 C CNN "Description"
+F 5 "Wurth Elektronik " H 6475 4250 50  0001 C CNN "MFN"
+F 6 "150080GS75000 " H 6475 4250 50  0001 C CNN "MFP"
+F 7 "https://www.mouser.com/ProductDetail/Wurth-Elektronik/150080GS75000?qs=2kOmHSv6VfQRoTEZVk1mGA%3D%3D" H 6475 4250 50  0001 C CNN "S1PL"
+F 8 " 710-150080GS75000 " H 6475 4250 50  0001 C CNN "S1PN"
 	1    6475 4250
 	0    1    -1   0
@@
 F 1 "YELLOW" V 6873 4330 50  0000 L CNN
 F 2 "LED_SMD:LED_0805_2012Metric_Pad1.15x1.40mm_HandSolder" H 6925 4250 50  0001 C CNN
-F 3 "~" H 6925 4250 50  0001 C CNN
+F 3 "https://www.mouser.com/datasheet/2/445/150080YS75000-1715432.pdf" H 6925 4250 50  0001 C CNN
+F 4 "Standard LEDs - SMD WL-SMCW SMDMono TpVw Waterclr 0805 Yellow " H 6925 4250 50  0001 C CNN "Description"
+F 5 "Wurth Elektronik " H 6925 4250 50  0001 C CNN "MFN"
+F 6 "150080YS75000" H 6925 4250 50  0001 C CNN "MFP"
+F 7 "https://www.mouser.com/ProductDetail/Wurth-Elektronik/150080YS75000?qs=LlUlMxKIyB3k0fZGrDMI2w%3D%3D" H 6925 4250 50  0001 C CNN "S1PL"
+F 8 " 710-150080YS75000 " H 6925 4250 50  0001 C CNN "S1PN"
 	1    6925 4250
 	0    1    -1   0
@@
 F 1 "YELLOW" V 7348 4330 50  0000 L CNN
 F 2 "LED_SMD:LED_0805_2012Metric_Pad1.15x1.40mm_HandSolder" H 7400 4250 50  0001 C CNN
-F 3 "~" H 7400 4250 50  0001 C CNN
+F 3 "https://www.mouser.com/datasheet/2/445/150080YS75000-1715432.pdf" H 7400 4250 50  0001 C CNN
+F 4 "Standard LEDs - SMD WL-SMCW SMDMono TpVw Waterclr 0805 Yellow " H 7400 4250 50  0001 C CNN "Description"
+F 5 "Wurth Elektronik " H 7400 4250 50  0001 C CNN "MFN"
+F 6 "150080YS75000" H 7400 4250 50  0001 C CNN "MFP"
+F 7 "https://www.mouser.com/ProductDetail/Wurth-Elektronik/150080YS75000?qs=LlUlMxKIyB3k0fZGrDMI2w%3D%3D" H 7400 4250 50  0001 C CNN "S1PL"
+F 8 " 710-150080YS75000 " H 7400 4250 50  0001 C CNN "S1PN"
 	1    7400 4250
 	0    1    -1   0
@@
 F 1 "YELLOW" V 7823 4330 50  0000 L CNN
 F 2 "LED_SMD:LED_0805_2012Metric_Pad1.15x1.40mm_HandSolder" H 7875 4250 50  0001 C CNN
-F 3 "~" H 7875 4250 50  0001 C CNN
+F 3 "https://www.mouser.com/datasheet/2/445/150080YS75000-1715432.pdf" H 7875 4250 50  0001 C CNN
+F 4 "Standard LEDs - SMD WL-SMCW SMDMono TpVw Waterclr 0805 Yellow " H 7875 4250 50  0001 C CNN "Description"
+F 5 "Wurth Elektronik " H 7875 4250 50  0001 C CNN "MFN"
+F 6 "150080YS75000" H 7875 4250 50  0001 C CNN "MFP"
+F 7 "https://www.mouser.com/ProductDetail/Wurth-Elektronik/150080YS75000?qs=LlUlMxKIyB3k0fZGrDMI2w%3D%3D" H 7875 4250 50  0001 C CNN "S1PL"
+F 8 " 710-150080YS75000 " H 7875 4250 50  0001 C CNN "S1PN"
 	1    7875 4250
 	0    1    -1   0
@@
 F 1 "GREEN" V 5698 4355 50  0000 L CNN
 F 2 "LED_SMD:LED_0805_2012Metric_Pad1.15x1.40mm_HandSolder" H 5750 4275 50  0001 C CNN
-F 3 "~" H 5750 4275 50  0001 C CNN
+F 3 "https://www.mouser.com/datasheet/2/445/150080GS75000-1715657.pdf" H 5750 4275 50  0001 C CNN
+F 4 "Standard LEDs - SMD WL-SMCW SMDMono TpVw Waterclr 0805 Green " H 5750 4275 50  0001 C CNN "Description"
+F 5 "Wurth Elektronik " H 5750 4275 50  0001 C CNN "MFN"
+F 6 "150080GS75000 " H 5750 4275 50  0001 C CNN "MFP"
+F 7 "https://www.mouser.com/ProductDetail/Wurth-Elektronik/150080GS75000?qs=2kOmHSv6VfQRoTEZVk1mGA%3D%3D" H 5750 4275 50  0001 C CNN "S1PL"
+F 8 " 710-150080GS75000 " H 5750 4275 50  0001 C CNN "S1PN"
 	1    5750 4275
 	0    1    -1   0
@@
 F 1 "BLUE" H 9018 5151 50  0000 C CNN
 F 2 "LED_SMD:LED_0805_2012Metric_Pad1.15x1.40mm_HandSolder" H 9025 5025 50  0001 C CNN
-F 3 "~" H 9025 5025 50  0001 C CNN
+F 3 "https://www.mouser.com/datasheet/2/445/150080BS75000-1715853.pdf" H 9025 5025 50  0001 C CNN
+F 4 "Standard LEDs - SMD WL-SMCW SMDMono TpVw Waterclr 0805 Blue " H 9025 5025 50  0001 C CNN "Description"
+F 5 "Wurth Elektronik " H 9025 5025 50  0001 C CNN "MFN"
+F 6 "150080BS75000 " H 9025 5025 50  0001 C CNN "MFP"
+F 7 "https://www.mouser.com/ProductDetail/Wurth-Elektronik/150080BS75000?qs=2kOmHSv6VfT2tBo3UPVqAQ%3D%3D" H 9025 5025 50  0001 C CNN "S1PL"
+F 8 " 710-150080BS75000 " H 9025 5025 50  0001 C CNN "S1PN"
 	1    9025 5025
 	-1   0    0    -1
@@
 F 1 "BLUE" H 9043 6676 50  0000 C CNN
 F 2 "LED_SMD:LED_0805_2012Metric_Pad1.15x1.40mm_HandSolder" H 9050 6550 50  0001 C CNN
-F 3 "~" H 9050 6550 50  0001 C CNN
+F 3 "https://www.mouser.com/datasheet/2/445/150080BS75000-1715853.pdf" H 9050 6550 50  0001 C CNN
+F 4 "Standard LEDs - SMD WL-SMCW SMDMono TpVw Waterclr 0805 Blue " H 9050 6550 50  0001 C CNN "Description"
+F 5 "Wurth Elektronik " H 9050 6550 50  0001 C CNN "MFN"
+F 6 "150080BS75000 " H 9050 6550 50  0001 C CNN "MFP"
+F 7 "https://www.mouser.com/ProductDetail/Wurth-Elektronik/150080BS75000?qs=2kOmHSv6VfT2tBo3UPVqAQ%3D%3D" H 9050 6550 50  0001 C CNN "S1PL"
+F 8 " 710-150080BS75000 " H 9050 6550 50  0001 C CNN "S1PN"
 	1    9050 6550
 	-1   0    0    -1
@@
 F 1 "YELLOW" V 12323 6155 50  0000 L CNN
 F 2 "LED_SMD:LED_0805_2012Metric_Pad1.15x1.40mm_HandSolder" H 12375 6075 50  0001 C CNN
-F 3 "~" H 12375 6075 50  0001 C CNN
+F 3 "https://www.mouser.com/datasheet/2/445/150080YS75000-1715432.pdf" H 12375 6075 50  0001 C CNN
+F 4 "Standard LEDs - SMD WL-SMCW SMDMono TpVw Waterclr 0805 Yellow " H 12375 6075 50  0001 C CNN "Description"
+F 5 "Wurth Elektronik " H 12375 6075 50  0001 C CNN "MFN"
+F 6 "150080YS75000" H 12375 6075 50  0001 C CNN "MFP"
+F 7 "https://www.mouser.com/ProductDetail/Wurth-Elektronik/150080YS75000?qs=LlUlMxKIyB3k0fZGrDMI2w%3D%3D" H 12375 6075 50  0001 C CNN "S1PL"
+F 8 " 710-150080YS75000 " H 12375 6075 50  0001 C CNN "S1PN"
 	1    12375 6075
 	0    1    -1   0
@@
 F 1 "YELLOW" V 15073 6180 50  0000 L CNN
 F 2 "LED_SMD:LED_0805_2012Metric_Pad1.15x1.40mm_HandSolder" H 15125 6100 50  0001 C CNN
-F 3 "~" H 15125 6100 50  0001 C CNN
+F 3 "https://www.mouser.com/datasheet/2/445/150080YS75000-1715432.pdf" H 15125 6100 50  0001 C CNN
+F 4 "Standard LEDs - SMD WL-SMCW SMDMono TpVw Waterclr 0805 Yellow " H 15125 6100 50  0001 C CNN "Description"
+F 5 "Wurth Elektronik " H 15125 6100 50  0001 C CNN "MFN"
+F 6 "150080YS75000" H 15125 6100 50  0001 C CNN "MFP"
+F 7 "https://www.mouser.com/ProductDetail/Wurth-Elektronik/150080YS75000?qs=LlUlMxKIyB3k0fZGrDMI2w%3D%3D" H 15125 6100 50  0001 C CNN "S1PL"
+F 8 " 710-150080YS75000 " H 15125 6100 50  0001 C CNN "S1PN"
 	1    15125 6100
 	0    1    -1   0
