File: pcb/main/pHMeter.sch (KiCad schematic (older format))
At the start: 90 parts, among them J1 Conn_02x03_Odd_Even, J4 AudioJack3_SwitchTR, J5 RJ12, J6 AudioJack3_SwitchTR, J7 SJ, Q1 ZXMS6004, Q2 ZXMS6004, Q3 DMP1045, Q4 ZXMS6004, Q5 ZXMS6004, SW1 Rotary_Encoder_Switch, U3 ATMEGA32U4-AU, U4 MCP1703A, U9 MCP73811T, X1 MINI-USB-SCHIELD-32005-201, Y1 Crystal

Commit message: perf: Replace folder libraries to lib_deps in platformio.ini. Previous performance: RAM:   [====      ]  39.1% (used 1001 bytes from 2560 bytes) Flash: [====      ]  40.2% (used 11518 bytes from 28672 bytes)
Current performance:
RAM:   [==        ]  23.5% (used 601 bytes from 2560 bytes)
Flash: [==        ]  22.5% (used 6460 bytes from 28672 bytes)
Parts:
- C6: value 100n -> 10u
- C7: value 10u -> 100n
Changed lines of the file:
@@
 P 2800 6575
 F 0 "C6" H 2915 6621 50  0000 L CNN
-F 1 "100n" H 2915 6530 50  0000 L CNN
+F 1 "10u" H 2915 6530 50  0000 L CNN
 F 2 "Capacitor_SMD:C_0805_2012Metric_Pad1.15x1.40mm_HandSolder" H 2838 6425 50  0001 C CNN
 F 3 "https://www.mouser.com/datasheet/2/445/885012207072-1727745.pdf" H 2800 6575 50  0001 C CNN
@@
 P 3175 6575
 F 0 "C7" H 3290 6621 50  0000 L CNN
-F 1 "10u" H 3290 6530 50  0000 L CNN
+F 1 "100n" H 3290 6530 50  0000 L CNN
 F 2 "Capacitor_SMD:C_0805_2012Metric_Pad1.15x1.40mm_HandSolder" H 3213 6425 50  0001 C CNN
 F 3 "https://www.mouser.com/datasheet/2/585/MLCC-1837944.pdf" H 3175 6575 50  0001 C CNN

Commit message: refactor: change conductometer circuit
Parts:
- removed D20: YELLOW, LED_SMD:LED_0805_2012Metric_Pad1.15x1.40mm_HandSolder, symbol Device:LED
- removed J6: AudioJack3_SwitchTR, Connector_Audio:Jack_3.5mm_Ledino_KB3SPRS_Horizontal, symbol Connector:AudioJack3_SwitchTR
- removed R50, R56: 1k, Resistor_SMD:R_0805_2012Metric_Pad1.15x1.40mm_HandSolder, symbol Device:R
- removed R52: 4.7k, Resistor_SMD:R_0805_2012Metric_Pad1.15x1.40mm_HandSolder, symbol Device:R
- removed R54: 100, Resistor_SMD:R_0805_2012Metric_Pad1.15x1.40mm_HandSolder, symbol Device:R
Connections:
- no-connect marks 10 -> 8
Changed lines of the file:
@@
 Sheet 1 6
 Title "PHMeter"
-Date "2021-05-09"
-Rev "0.2"
+Date "2021-11-26"
+Rev "0.3"
 Comp "Hackuarium"
 Comment1 "New version for pH and conductivity Meter"
@@
 F7 "MOSI" I R 4975 3975 50
 $EndSheet
-$Sheet
-S 700  4300 650  350
-U 5F3634CD
-F0 "Conductometer" 50
-F1 "Conductometer.sch" 50
-F2 "VIn" I L 700 4475 50
-F3 "VOut" I R 1350 4475 50
-$EndSheet
 Text GLabel 625  4400 1    50   Input ~ 0
 3.3V
@@
 	11000 6450 11100 6450
 $Comp
-L Device:R R56
-U 1 1 5F9CF052
-P 14900 5875
-F 0 "R56" V 14693 5875 50  0000 C CNN
-F 1 "1k" V 14784 5875 50  0000 C CNN
-F 2 "Resistor_SMD:R_0805_2012Metric_Pad1.15x1.40mm_HandSolder" V 14830 5875 50  0001 C CNN
-F 3 "~" H 14900 5875 50  0001 C CNN
-	1    14900 5875
-	0    1    1    0
-$EndComp
-$Comp
-L Device:R R54
-U 1 1 5F9CF058
-P 14675 6100
-F 0 "R54" H 14605 6054 50  0000 R CNN
-F 1 "100" H 14605 6145 50  0000 R CNN
-F 2 "Resistor_SMD:R_0805_2012Metric_Pad1.15x1.40mm_HandSolder" V 14605 6100 50  0001 C CNN
-F 3 "~" H 14675 6100 50  0001 C CNN
-	1    14675 6100
-	-1   0    0    1
-$EndComp
-Text GLabel 14600 5875 0    50   Input ~ 0
-3.3V
-Wire Wire Line
-	14600 5875 14675 5875
-Wire Wire Line
-	14675 5950 14675 5875
-Connection ~ 14675 5875
-Wire Wire Line
-	14675 5875 14750 5875
-Wire Wire Line
-	15050 5875 15125 5875
-Wire Wire Line
-	15125 5875 15125 5950
-Wire Wire Line
-	15125 6250 15125 6325
-Wire Wire Line
-	15125 6325 15200 6325
-Wire Wire Line
-	14675 6250 14675 6325
-Wire Wire Line
-	14675 6325 15125 6325
-Connection ~ 15125 6325
-$Comp
-L Device:R R52
-U 1 1 5F9CF06A
-P 14450 6325
-F 0 "R52" V 14657 6325 50  0000 C CNN
-F 1 "4.7k" V 14566 6325 50  0000 C CNN
-F 2 "Resistor_SMD:R_0805_2012Metric_Pad1.15x1.40mm_HandSolder" V 14380 6325 50  0001 C CNN
-F 3 "~" H 14450 6325 50  0001 C CNN
-	1    14450 6325
-	0    -1   -1   0
-$EndComp
-$Comp
-L Device:R R50
-U 1 1 5F9CF070
-P 14000 6475
-F 0 "R50" V 14207 6475 50  0000 C CNN
-F 1 "1k" V 14116 6475 50  0000 C CNN
-F 2 "Resistor_SMD:R_0805_2012Metric_Pad1.15x1.40mm_HandSolder" V 13930 6475 50  0001 C CNN
-F 3 "~" H 14000 6475 50  0001 C CNN
-	1    14000 6475
-	0    -1   -1   0
-$EndComp
-Wire Wire Line
-	14600 6325 14675 6325
-Connection ~ 14675 6325
-$Comp
-L Bertha_main-eagle-import:GND #U06
-U 1 1 5F9CF078
-P 14675 6900
-F 0 "#U06" H 14725 6950 50  0001 C CNN
-F 1 "GND" H 14778 6938 42  0000 L CNN
-F 2 "" H 14675 6900 50  0001 C CNN
-F 3 "" H 14675 6900 50  0001 C CNN
-	1    14675 6900
-	1    0    0    -1
-$EndComp
-Wire Wire Line
-	15200 6425 14675 6425
-Wire Wire Line
-	14675 6425 14675 6800
-NoConn ~ 15200 6525
-NoConn ~ 15200 6725
-Wire Wire Line
-	15200 6625 14225 6625
-Wire Wire Line
-	14225 6625 14225 6475
-Wire Wire Line
-	14225 6325 14300 6325
-Wire Wire Line
-	14150 6475 14225 6475
-Connection ~ 14225 6475
-Wire Wire Line
-	14225 6475 14225 6325
-Text GLabel 13750 6475 0    50   Input ~ 0
-D7
-Wire Wire Line
-	13750 6475 13850 6475
-$Comp
 L Connector:AudioJack3_SwitchTR J4
 U 1 1 5FA04BCE
@@
 F 3 "~" H 12650 6400 50  0001 C CNN
 	1    12650 6400
-	-1   0    0    -1
-$EndComp
-$Comp
-L Connector:AudioJack3_SwitchTR J6
-U 1 1 5FA2F68F
-P 15400 6425
-F 0 "J6" V 15100 6325 50  0000 R CNN
-F 1 "AudioJack3_SwitchTR" V 15025 6725 50  0000 R CNN
-F 2 "Connector_Audio:Jack_3.5mm_Ledino_KB3SPRS_Horizontal" H 15400 6425 50  0001 C CNN
-F 3 "~" H 15400 6425 50  0001 C CNN
-	1    15400 6425
 	-1   0    0    -1
 $EndComp
@@
 	0    1    -1   0
 $EndComp
-$Comp
-L Device:LED D20
-U 1 1 5FA5C1EC
-P 15125 6100
-F 0 "D20" V 15164 6180 50  0000 L CNN
-F 1 "YELLOW" V 15073 6180 50  0000 L CNN
-F 2 "LED_SMD:LED_0805_2012Metric_Pad1.15x1.40mm_HandSolder" H 15125 6100 50  0001 C CNN
-F 3 "https://www.mouser.com/datasheet/2/445/150080YS75000-1715432.pdf" H 15125 6100 50  0001 C CNN
-F 4 "Standard LEDs - SMD WL-SMCW SMDMono TpVw Waterclr 0805 Yellow " H 15125 6100 50  0001 C CNN "Description"
-F 5 "Wurth Elektronik " H 15125 6100 50  0001 C CNN "MFN"
-F 6 "150080YS75000" H 15125 6100 50  0001 C CNN "MFP"
-F 7 "https://www.mouser.com/ProductDetail/Wurth-Elektronik/150080YS75000?qs=LlUlMxKIyB3k0fZGrDMI2w%3D%3D" H 15125 6100 50  0001 C CNN "S1PL"
-F 8 " 710-150080YS75000 " H 15125 6100 50  0001 C CNN "S1PN"
-	1    15125 6100
-	0    1    -1   0
-$EndComp
 Text GLabel 5425 9775 0    50   Input ~ 0
 RX
@@
 Text Notes 6250 4875 1    50   ~ 0
 Power LED for 3.3 V is place into 3.sch.
+$Sheet
+S 700  4325 650  300
+U 61A4519E
+F0 "Conductometer_2" 50
+F1 "Conductometer_2.sch" 50
+F2 "Vout" I R 1350 4475 50
+F3 "Vin" I L 700 4475 50
+$EndSheet
 $EndSCHEMATC

Commit message: build: pHMeter version 0.2
Add new circuit for conductometer.
Parts:
- removed D10: YELLOW, LED_SMD:LED_0805_2012Metric_Pad1.15x1.40mm_HandSolder, symbol Device:LED
- added J6: AudioJack3_SwitchTR, Connector_Audio:Jack_3.5mm_Ledino_KB3SPRS_Horizontal, symbol Connector:AudioJack3_SwitchTR
- added R19: 1k, Resistor_SMD:R_0805_2012Metric_Pad1.15x1.40mm_HandSolder, symbol Device:R
- added R22: 100, Resistor_SMD:R_0805_2012Metric_Pad1.15x1.40mm_HandSolder, symbol Device:R
- R21: value 1k -> 4.7k
Connections:
- net +3V3: now also R23.2, R22.2; no longer R21.1, R23.1
- net A5: no longer R29.1, R30.2
- net D7: no longer R49.1
- net at D9.2 (A): now also R23.1; no longer R21.2
- net RXLED: no longer names the net of D9.1 (K)
- net RXLED: now also R21.2, J6.S, R22.1; no longer U3.8 (PB0(SS))
- net TXLED renamed ONE-WIRE-2
- net ONE-WIRE-2: now also R19.1
- new net: R29.1, R30.2
- new net: J6.T, R19.2, R21.1
- new net ONE-WIRE-1: R49.1, U3.8 (PB0(SS))
- no-connect marks 8 -> 10
Changed lines of the file:
@@
-	1    0    0    -1
-$EndComp
-$Comp
-L Device:R R23
-U 1 1 5EDC8DAC
-P 7400 3850
-F 0 "R23" H 7470 3896 50  0000 L CNN
-F 1 "1k" H 7470 3805 50  0000 L CNN
-F 2 "Resistor_SMD:R_0805_2012Metric_Pad1.15x1.40mm_HandSolder" V 7330 3850 50  0001 C CNN
-F 3 "~" H 7400 3850 50  0001 C CNN
-	1    7400 3850
 	1    0    0    -1
 $EndComp
@@
 	7875 3700 7875 3600
 Wire Wire Line
-	7400 3700 7400 3600
-Wire Wire Line
 	7875 4000 7875 4100
-Wire Wire Line
-	7400 4000 7400 4100
-Text GLabel 7400 4500 3    50   Input ~ 0
-TXLED
 Text GLabel 7875 4500 3    50   Input ~ 0
 TX
 Wire Wire Line
 	7875 4400 7875 4500
-Wire Wire Line
-	7400 4400 7400 4500
 Text GLabel 3500 4000 2    50   Input ~ 0
 A0
@@
 Text GLabel 7875 3600 1    50   Input ~ 0
 3.3V
-Text GLabel 7400 3600 1    50   Input ~ 0
-3.3V
 Text GLabel 5250 5850 2    50   Input ~ 0
 VUSB
@@
 Text Notes 6925 3175 0    100  ~ 0
 COM LEDs
-Text GLabel 6925 3600 1    50   Input ~ 0
-3.3V
-Wire Wire Line
-	6925 4400 6925 4500
-Text GLabel 6925 4500 3    50   Input ~ 0
-RXLED
-Wire Wire Line
-	6925 4100 6925 4000
-Wire Wire Line
-	6925 3600 6925 3700
-$Comp
-L Device:R R21
-U 1 1 5EDC90A6
-P 6925 3850
-F 0 "R21" H 6995 3896 50  0000 L CNN
-F 1 "1k" H 6995 3805 50  0000 L CNN
-F 2 "Resistor_SMD:R_0805_2012Metric_Pad1.15x1.40mm_HandSolder" V 6855 3850 50  0001 C CNN
-F 3 "~" H 6925 3850 50  0001 C CNN
-	1    6925 3850
-	1    0    0    -1
-$EndComp
 Wire Wire Line
 	6475 4400 6475 4500
@@
 F 8 " 710-150080GS75000 " H 6475 4250 50  0001 C CNN "S1PN"
 	1    6475 4250
-	0    1    -1   0
-$EndComp
-$Comp
-L Device:LED D9
-U 1 1 5EE57147
-P 6925 4250
-F 0 "D9" V 6964 4330 50  0000 L CNN
-F 1 "YELLOW" V 6873 4330 50  0000 L CNN
-F 2 "LED_SMD:LED_0805_2012Metric_Pad1.15x1.40mm_HandSolder" H 6925 4250 50  0001 C CNN
-F 3 "https://www.mouser.com/datasheet/2/445/150080YS75000-1715432.pdf" H 6925 4250 50  0001 C CNN
-F 4 "Standard LEDs - SMD WL-SMCW SMDMono TpVw Waterclr 0805 Yellow " H 6925 4250 50  0001 C CNN "Description"
-F 5 "Wurth Elektronik " H 6925 4250 50  0001 C CNN "MFN"
-F 6 "150080YS75000" H 6925 4250 50  0001 C CNN "MFP"
-F 7 "https://www.mouser.com/ProductDetail/Wurth-Elektronik/150080YS75000?qs=LlUlMxKIyB3k0fZGrDMI2w%3D%3D" H 6925 4250 50  0001 C CNN "S1PL"
-F 8 " 710-150080YS75000 " H 6925 4250 50  0001 C CNN "S1PN"
-	1    6925 4250
-	0    1    -1   0
-$EndComp
-$Comp
-L Device:LED D10
-U 1 1 5EE5769A
-P 7400 4250
-F 0 "D10" V 7439 4330 50  0000 L CNN
-F 1 "YELLOW" V 7348 4330 50  0000 L CNN
-F 2 "LED_SMD:LED_0805_2012Metric_Pad1.15x1.40mm_HandSolder" H 7400 4250 50  0001 C CNN
-F 3 "https://www.mouser.com/datasheet/2/445/150080YS75000-1715432.pdf" H 7400 4250 50  0001 C CNN
-F 4 "Standard LEDs - SMD WL-SMCW SMDMono TpVw Waterclr 0805 Yellow " H 7400 4250 50  0001 C CNN "Description"
-F 5 "Wurth Elektronik " H 7400 4250 50  0001 C CNN "MFN"
-F 6 "150080YS75000" H 7400 4250 50  0001 C CNN "MFP"
-F 7 "https://www.mouser.com/ProductDetail/Wurth-Elektronik/150080YS75000?qs=LlUlMxKIyB3k0fZGrDMI2w%3D%3D" H 7400 4250 50  0001 C CNN "S1PL"
-F 8 " 710-150080YS75000 " H 7400 4250 50  0001 C CNN "S1PN"
-	1    7400 4250
 	0    1    -1   0
 $EndComp
@@
 Text GLabel 14450 3450 2    50   Input ~ 0
 SCK
-Text GLabel 14450 3550 2    50   Input ~ 0
-RXLED
 Text GLabel 14450 3750 2    50   Input ~ 0
 D6
 Text GLabel 14450 3850 2    50   Input ~ 0
 D12
-Text GLabel 14450 3950 2    50   Input ~ 0
-TXLED
 Text GLabel 14450 4050 2    50   Input ~ 0
 A6
@@
 	14450 3450 14300 3450
 Wire Wire Line
-	14300 3550 14450 3550
-Wire Wire Line
 	14450 3750 14300 3750
 Wire Wire Line
 	14300 3850 14450 3850
-Wire Wire Line
-	14450 3950 14300 3950
 Wire Wire Line
 	14300 4050 14450 4050
@@
 Wire Wire Line
 	625  4475 700  4475
-Text GLabel 1450 4475 2    50   Input ~ 0
-A+
 Wire Wire Line
 	1450 4475 1350 4475
@@
 	650  2275 650  2150
 Wire Wire Line
-	1025 1775 1100 1775
-Wire Wire Line
-	1100 1775 1100 1600
-Connection ~ 1100 1775
-Wire Wire Line
-	1100 1775 1250 1775
-Text GLabel 1100 1600 1    50   Input ~ 0
-A5
-Wire Wire Line
 	650  1675 650  1775
 Text GLabel 2125 1500 1    50   Input ~ 0
@@
 	11475 6450 11475 6300
 Text GLabel 11000 6450 0    50   Input ~ 0
-D7
+ONE-WIRE-1
 Wire Wire Line
 	11000 6450 11100 6450
@@
 F3 "Vin" I L 700 4475 50
 $EndSheet
+Wire Wire Line
+	1025 1775 1250 1775
+Text GLabel 1450 4475 2    50   Input ~ 0
+A5
+$Comp
+L Device:R R23
+U 1 1 61B59881
+P 14875 5825
+F 0 "R23" V 14668 5825 50  0000 C CNN
+F 1 "1k" V 14759 5825 50  0000 C CNN
+F 2 "Resistor_SMD:R_0805_2012Metric_Pad1.15x1.40mm_HandSolder" V 14805 5825 50  0001 C CNN
+F 3 "~" H 14875 5825 50  0001 C CNN
+	1    14875 5825
+	0    1    1    0
+$EndComp
+$Comp
+L Device:R R22
+U 1 1 61B59E35
+P 14650 6050
+F 0 "R22" H 14580 6004 50  0000 R CNN
+F 1 "100" H 14580 6095 50  0000 R CNN
+F 2 "Resistor_SMD:R_0805_2012Metric_Pad1.15x1.40mm_HandSolder" V 14580 6050 50  0001 C CNN
+F 3 "~" H 14650 6050 50  0001 C CNN
+	1    14650 6050
+	-1   0    0    1
+$EndComp
+$Comp
+L Device:LED D9
+U 1 1 61B5AB1F
+P 15100 6050
+F 0 "D9" V 15139 6130 50  0000 L CNN
+F 1 "YELLOW" V 15048 6130 50  0000 L CNN
+F 2 "LED_SMD:LED_0805_2012Metric_Pad1.15x1.40mm_HandSolder" H 15100 6050 50  0001 C CNN
+F 3 "https://www.mouser.com/datasheet/2/445/150080YS75000-1715432.pdf" H 15100 6050 50  0001 C CNN
+F 4 "Standard LEDs - SMD WL-SMCW SMDMono TpVw Waterclr 0805 Yellow " H 15100 6050 50  0001 C CNN "Description"
+F 5 "Wurth Elektronik " H 15100 6050 50  0001 C CNN "MFN"
+F 6 "150080YS75000" H 15100 6050 50  0001 C CNN "MFP"
+F 7 "https://www.mouser.com/ProductDetail/Wurth-Elektronik/150080YS75000?qs=LlUlMxKIyB3k0fZGrDMI2w%3D%3D" H 15100 6050 50  0001 C CNN "S1PL"
+F 8 " 710-150080YS75000 " H 15100 6050 50  0001 C CNN "S1PN"
+	1    15100 6050
+	0    1    -1   0
+$EndComp
+$Comp
+L Connector:AudioJack3_SwitchTR J6
+U 1 1 61B5B879
+P 15400 6400
+F 0 "J6" V 15100 6300 50  0000 R CNN
+F 1 "AudioJack3_SwitchTR" V 15025 6650 50  0000 R CNN
+F 2 "Connector_Audio:Jack_3.5mm_Ledino_KB3SPRS_Horizontal" H 15400 6400 50  0001 C CNN
+F 3 "~" H 15400 6400 50  0001 C CNN
+	1    15400 6400
+	-1   0    0    -1
+$EndComp
+$Comp
+L Device:R R21
+U 1 1 61B5D37C
+P 14425 6300
+F 0 "R21" V 14632 6300 50  0000 C CNN
+F 1 "4.7k" V 14541 6300 50  0000 C CNN
+F 2 "Resistor_SMD:R_0805_2012Metric_Pad1.15x1.40mm_HandSolder" V 14355 6300 50  0001 C CNN
+F 3 "~" H 14425 6300 50  0001 C CNN
+	1    14425 6300
+	0    -1   -1   0
+$EndComp
+$Comp
+L Device:R R19
+U 1 1 61B5DB7D
+P 13975 6450
+F 0 "R19" V 14182 6450 50  0000 C CNN
+F 1 "1k" V 14091 6450 50  0000 C CNN
+F 2 "Resistor_SMD:R_0805_2012Metric_Pad1.15x1.40mm_HandSolder" V 13905 6450 50  0001 C CNN
+F 3 "~" H 13975 6450 50  0001 C CNN
+	1    13975 6450
+	0    -1   -1   0
+$EndComp
+Wire Wire Line
+	14575 6300 14650 6300
+Wire Wire Line
+	14650 6300 14650 6200
+Wire Wire Line
+	14650 5900 14650 5825
+Wire Wire Line
+	14650 5825 14725 5825
+Wire Wire Line
+	15025 5825 15100 5825
+Wire Wire Line
+	15100 5825 15100 5900
+NoConn ~ 15200 6500
+NoConn ~ 15200 6700
+Wire Wire Line
+	14650 6300 15100 6300
+Connection ~ 14650 6300
+Wire Wire Line
+	15100 6200 15100 6300
+Connection ~ 15100 6300
+Wire Wire Line
+	15100 6300 15200 6300
+Text GLabel 14575 5825 0    50   Input ~ 0
+3.3V
+Wire Wire Line
+	14575 5825 14650 5825
+Connection ~ 14650 5825
+Wire Wire Line
+	14125 6450 14200 6450
+Wire Wire Line
+	14200 6450 14200 6300
+Wire Wire Line
+	14200 6300 14275 6300
+Wire Wire Line
+	15200 6600 14200 6600
+Wire Wire Line
+	14200 6600 14200 6450
+Connection ~ 14200 6450
+$Comp
+L Bertha_main-eagle-import:GND #U0106
+U 1 1 61CD0E6E
+P 14650 6875
+F 0 "#U0106" H 14700 6925 50  0001 C CNN
+F 1 "GND" H 14753 6913 42  0000 L CNN
+F 2 "" H 14650 6875 50  0001 C CNN
+F 3 "" H 14650 6875 50  0001 C CNN
+	1    14650 6875
+	1    0    0    -1
+$EndComp
+Wire Wire Line
+	14650 6775 14650 6400
+Wire Wire Line
+	14650 6400 15200 6400
+Text GLabel 14450 3550 2    50   Input ~ 0
+ONE-WIRE-1
+Text GLabel 14450 3950 2    50   Input ~ 0
+ONE-WIRE-2
+Wire Wire Line
+	14450 3950 14300 3950
+Wire Wire Line
+	14450 3550 14300 3550
+Text GLabel 13725 6450 0    50   Input ~ 0
+ONE-WIRE-2
+Wire Wire Line
+	13725 6450 13825 6450
 $EndSCHEMATC
