File: pcb/main/3.sch (KiCad schematic (older format))
At the start: 10 parts, among them U5 AP63203WU-7

Commit message: Fix: renamed value for LEDs
Parts:
- C19: Description (none) -> Multilayer Ceramic Capacitors MLCC - SMD/SMT 16V 10uF X5R 0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; MFN (none) -> Samsung Electro-Mechanics; MFP (none) -> CL21A106KOQNNNG; S1PL (none) -> https://www.mouser.com/ProductDetail/Samsung-Electro-Mechan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; S1PN (none) -> 187-CL21A106KOQNNNG
- C22: Description (none) -> Multilayer Ceramic Capacitors MLCC - SMD/SMT WCAP-CSGP 0.1u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; MFN (none) -> Wurth Elektronik; MFP (none) -> 885012207072; S1PL (none) -> https://www.mouser.com/ProductDetail/Wurth-Elektronik/88501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; S1PN (none) -> 710-885012207072
- C24, C25: Description (none) -> Multilayer Ceramic Capacitors MLCC - SMD/SMT 6.3V 22uF X5R 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; MFN (none) -> Samsung Electro-Mechanics; MFP (none) -> CL21A226KQCLRNC; S1PL (none) -> https://www.mouser.com/ProductDetail/Samsung-Electro-Mechan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; S1PN (none) -> 187-CL21A226KQCLRNC
- D15, D16: value RED -> GREEN
- L2: footprint Inductor_SMD:L_TDK_SLF6028 -> Inductor_SMD:L_Taiyo-Yuden_NR-40xx_HandSoldering
Changed lines of the file:
@@
 P 6850 4175
 F 0 "D15" H 6850 4100 50  0000 C CNN
-F 1 "RED" H 6850 4275 50  0000 C CNN
+F 1 "GREEN" H 6850 4275 50  0000 C CNN
 F 2 "LED_SMD:LED_0805_2012Metric_Pad1.15x1.40mm_HandSolder" H 6850 4175 50  0001 C CNN
 F 3 "~" H 6850 4175 50  0001 C CNN
@@
 P 7450 4175
 F 0 "D16" H 7450 4100 50  0000 C CNN
-F 1 "RED" H 7450 4275 50  0000 C CNN
+F 1 "GREEN" H 7450 4275 50  0000 C CNN
 F 2 "LED_SMD:LED_0805_2012Metric_Pad1.15x1.40mm_HandSolder" H 7450 4175 50  0001 C CNN
 F 3 "~" H 7450 4175 50  0001 C CNN
@@
 F 1 "10u" H 3465 3905 50  0000 L CNN
 F 2 "Capacitor_SMD:C_0805_2012Metric_Pad1.15x1.40mm_HandSolder" H 3388 3800 50  0001 C CNN
-F 3 "~" H 3350 3950 50  0001 C CNN
+F 3 "https://www.mouser.com/datasheet/2/585/MLCC-1837944.pdf" H 3350 3950 50  0001 C CNN
+F 4 "Multilayer Ceramic Capacitors MLCC - SMD/SMT 16V 10uF X5R 0805 10%" H 3350 3950 50  0001 C CNN "Description"
+F 5 "Samsung Electro-Mechanics " H 3350 3950 50  0001 C CNN "MFN"
+F 6 "CL21A106KOQNNNG " H 3350 3950 50  0001 C CNN "MFP"
+F 7 "https://www.mouser.com/ProductDetail/Samsung-Electro-Mechanics/CL21A106KOQNNNG?qs=hqM3L16%252BxlcMWI7QbqH0LA%3D%3D" H 3350 3950 50  0001 C CNN "S1PL"
+F 8 " 187-CL21A106KOQNNNG " H 3350 3950 50  0001 C CNN "S1PN"
 	1    3350 3950
 	1    0    0    -1
@@
 F 1 "100n" V 4539 3850 50  0000 C CNN
 F 2 "Capacitor_SMD:C_0805_2012Metric_Pad1.15x1.40mm_HandSolder" H 4738 3700 50  0001 C CNN
-F 3 "~" H 4700 3850 50  0001 C CNN
+F 3 "https://www.mouser.com/datasheet/2/445/885012207072-1727745.pdf" H 4700 3850 50  0001 C CNN
+F 4 "Multilayer Ceramic Capacitors MLCC - SMD/SMT WCAP-CSGP 0.1uF 0805 10% 25V MLCC " H 4700 3850 50  0001 C CNN "Description"
+F 5 "Wurth Elektronik " H 4700 3850 50  0001 C CNN "MFN"
+F 6 "885012207072" H 4700 3850 50  0001 C CNN "MFP"
+F 7 "https://www.mouser.com/ProductDetail/Wurth-Elektronik/885012207072?qs=0KOYDY2FL28rQMV4504TxA%3D%3D" H 4700 3850 50  0001 C CNN "S1PL"
+F 8 "710-885012207072 " H 4700 3850 50  0001 C CNN "S1PN"
 	1    4700 3850
 	0    1    1    0
@@
 F 0 "L2" V 5315 3750 50  0000 C CNN
 F 1 "3.9u" V 5224 3750 50  0000 C CNN
-F 2 "Inductor_SMD:L_TDK_SLF6028" H 5125 3750 50  0001 C CNN
+F 2 "Inductor_SMD:L_Taiyo-Yuden_NR-40xx_HandSoldering" H 5125 3750 50  0001 C CNN
 F 3 "~" H 5125 3750 50  0001 C CNN
 	1    5125 3750
@@
 F 1 "22u" H 5335 3995 50  0000 R CNN
 F 2 "Capacitor_SMD:C_0805_2012Metric_Pad1.15x1.40mm_HandSolder" H 5488 3800 50  0001 C CNN
-F 3 "~" H 5450 3950 50  0001 C CNN
+F 3 "https://www.mouser.com/datasheet/2/585/MLCC-1837944.pdf" H 5450 3950 50  0001 C CNN
+F 4 "Multilayer Ceramic Capacitors MLCC - SMD/SMT 6.3V 22uF X5R 10% 0805" H 5450 3950 50  0001 C CNN "Description"
+F 5 "Samsung Electro-Mechanics " H 5450 3950 50  0001 C CNN "MFN"
+F 6 "CL21A226KQCLRNC" H 5450 3950 50  0001 C CNN "MFP"
+F 7 "https://www.mouser.com/ProductDetail/Samsung-Electro-Mechanics/CL21A226KQCLRNC?qs=xZ%2FP%252Ba9zWqYG0ePGTF%2FymQ%3D%3D" H 5450 3950 50  0001 C CNN "S1PL"
+F 8 " 187-CL21A226KQCLRNC " H 5450 3950 50  0001 C CNN "S1PN"
 	1    5450 3950
 	-1   0    0    1
@@
 F 1 "22u" H 5685 3995 50  0000 R CNN
 F 2 "Capacitor_SMD:C_0805_2012Metric_Pad1.15x1.40mm_HandSolder" H 5838 3800 50  0001 C CNN
-F 3 "~" H 5800 3950 50  0001 C CNN
+F 3 "https://www.mouser.com/datasheet/2/585/MLCC-1837944.pdf" H 5800 3950 50  0001 C CNN
+F 4 "Multilayer Ceramic Capacitors MLCC - SMD/SMT 6.3V 22uF X5R 10% 0805" H 5800 3950 50  0001 C CNN "Description"
+F 5 "Samsung Electro-Mechanics " H 5800 3950 50  0001 C CNN "MFN"
+F 6 "CL21A226KQCLRNC" H 5800 3950 50  0001 C CNN "MFP"
+F 7 "https://www.mouser.com/ProductDetail/Samsung-Electro-Mechanics/CL21A226KQCLRNC?qs=xZ%2FP%252Ba9zWqYG0ePGTF%2FymQ%3D%3D" H 5800 3950 50  0001 C CNN "S1PL"
+F 8 " 187-CL21A226KQCLRNC " H 5800 3950 50  0001 C CNN "S1PN"
 	1    5800 3950
 	-1   0    0    1

Commit message: Fix: Changed BNC connector for pH and conductometer (issue #3)
Parts:
- D15, D16: Description (none) -> Standard LEDs - SMD WL-SMCW SMDMono TpVw Waterclr 0805 Green; MFN (none) -> Wurth Elektronik; MFP (none) -> 150080GS75000; S1PL (none) -> https://www.mouser.com/ProductDetail/Wurth-Elektronik/15008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; S1PN (none) -> 710-150080GS75000
Changed lines of the file:
@@
 F 1 "GREEN" H 6850 4275 50  0000 C CNN
 F 2 "LED_SMD:LED_0805_2012Metric_Pad1.15x1.40mm_HandSolder" H 6850 4175 50  0001 C CNN
-F 3 "~" H 6850 4175 50  0001 C CNN
+F 3 "https://www.mouser.com/datasheet/2/445/150080GS75000-1715657.pdf" H 6850 4175 50  0001 C CNN
+F 4 "Standard LEDs - SMD WL-SMCW SMDMono TpVw Waterclr 0805 Green " H 6850 4175 50  0001 C CNN "Description"
+F 5 "Wurth Elektronik " H 6850 4175 50  0001 C CNN "MFN"
+F 6 "150080GS75000 " H 6850 4175 50  0001 C CNN "MFP"
+F 7 "https://www.mouser.com/ProductDetail/Wurth-Elektronik/150080GS75000?qs=2kOmHSv6VfQRoTEZVk1mGA%3D%3D" H 6850 4175 50  0001 C CNN "S1PL"
+F 8 " 710-150080GS75000 " H 6850 4175 50  0001 C CNN "S1PN"
 	1    6850 4175
 	0    1    -1   0
@@
 F 1 "GREEN" H 7450 4275 50  0000 C CNN
 F 2 "LED_SMD:LED_0805_2012Metric_Pad1.15x1.40mm_HandSolder" H 7450 4175 50  0001 C CNN
-F 3 "~" H 7450 4175 50  0001 C CNN
+F 3 "https://www.mouser.com/datasheet/2/445/150080GS75000-1715657.pdf" H 7450 4175 50  0001 C CNN
+F 4 "Standard LEDs - SMD WL-SMCW SMDMono TpVw Waterclr 0805 Green " H 7450 4175 50  0001 C CNN "Description"
+F 5 "Wurth Elektronik " H 7450 4175 50  0001 C CNN "MFN"
+F 6 "150080GS75000 " H 7450 4175 50  0001 C CNN "MFP"
+F 7 "https://www.mouser.com/ProductDetail/Wurth-Elektronik/150080GS75000?qs=2kOmHSv6VfQRoTEZVk1mGA%3D%3D" H 7450 4175 50  0001 C CNN "S1PL"
+F 8 " 710-150080GS75000 " H 7450 4175 50  0001 C CNN "S1PN"
 	1    7450 4175
 	0    1    -1   0

Commit message: build: pHMeter version 0.2
Add new circuit for conductometer.
Parts:
- L2: footprint Inductor_SMD:L_Taiyo-Yuden_NR-40xx_HandSoldering -> Inductor_SMD:L_Taiyo-Yuden_NR-24xx_HandSoldering
Changed lines of the file:
@@
 F 0 "L2" V 5315 3750 50  0000 C CNN
 F 1 "3.9u" V 5224 3750 50  0000 C CNN
-F 2 "Inductor_SMD:L_Taiyo-Yuden_NR-40xx_HandSoldering" H 5125 3750 50  0001 C CNN
+F 2 "Inductor_SMD:L_Taiyo-Yuden_NR-24xx_HandSoldering" H 5125 3750 50  0001 C CNN
 F 3 "~" H 5125 3750 50  0001 C CNN
 	1    5125 3750
