File: pcb/main/Conductometer_2.sch (KiCad schematic (older format))
At the start: 30 parts, among them J2 Conn_Coaxial_Power, U10 LM2660M, U2 TLV6004PW, U8 CD4060BM

Commit message: fix: solve CD4060BM and LM2660M fingerprints
Original fingerprint from manufacturer has an inconsistent desing.
Parts:
- U10: footprint LM2060M:LM2660M -> pHMeter:LM2660M
- U8: footprint CD4060BM:CD4060BM -> pHMeter:CD4060BM; symbol CD4060BM:CD4060BM -> pHMeter-rescue:CD4060BM-CD4060BM
Changed lines of the file:
@@
 NoConn ~ 5425 5325
 $Comp
-L CD4060BM:CD4060BM U8
+L pHMeter-rescue:CD4060BM-CD4060BM U8
 U 1 1 61A4BEA9
 P 5425 4825
+AR Path="/61A4BEA9" Ref="U8"  Part="1"
+AR Path="/61A4519E/61A4BEA9" Ref="U8"  Part="1"
 F 0 "U8" H 6625 5212 60  0000 C CNN
 F 1 "CD4060BM" H 6625 5106 60  0000 C CNN
-F 2 "CD4060BM:CD4060BM" H 6625 5065 60  0001 C CNN
+F 2 "pHMeter:CD4060BM" H 6625 5065 60  0001 C CNN
 F 3 "" H 5425 4825 60  0000 C CNN
 	1    5425 4825
@@
 F 0 "U10" H 8775 1662 60  0000 C CNN
 F 1 "LM2660M" H 8775 1556 60  0000 C CNN
-F 2 "LM2060M:LM2660M" H 8775 1515 60  0001 C CNN
+F 2 "pHMeter:LM2660M" H 8775 1515 60  0001 C CNN
 F 3 "" H 7675 1275 60  0000 C CNN
 	1    7675 1275
