File: pcb/main/24bits ADC.sch (KiCad schematic (older format))
At the start: 9 parts, among them J8 SJ, U6 HX711

Commit message: Fix: renamed value for LEDs
Parts:
- C26, C28, C30: value 100nF -> 100n; Description (none) -> Multilayer Ceramic Capacitors MLCC - SMD/SMT WCAP-CSGP 0.1u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; MFN (none) -> Wurth Elektronik; MFP (none) -> 885012207072; S1PL (none) -> https://www.mouser.com/ProductDetail/Wurth-Elektronik/88501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; S1PN (none) -> 710-885012207072
- C27, C29: value 10uF -> 10u; Description (none) -> Multilayer Ceramic Capacitors MLCC - SMD/SMT 16V 10uF X5R 0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; MFN (none) -> Samsung Electro-Mechanics; MFP (none) -> CL21A106KOQNNNG; S1PL (none) -> https://www.mouser.com/ProductDetail/Samsung-Electro-Mechan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; S1PN (none) -> 187-CL21A106KOQNNNG
Changed lines of the file:
@@
 P 3800 4875
 F 0 "C26" H 3925 4925 50  0000 L CNN
-F 1 "100nF" H 3825 4775 50  0000 L CNN
+F 1 "100n" H 3825 4775 50  0000 L CNN
 F 2 "Capacitor_SMD:C_0805_2012Metric_Pad1.15x1.40mm_HandSolder" H 3838 4725 50  0001 C CNN
-F 3 "~" H 3800 4875 50  0001 C CNN
+F 3 "https://www.mouser.com/datasheet/2/445/885012207072-1727745.pdf" H 3800 4875 50  0001 C CNN
+F 4 "Multilayer Ceramic Capacitors MLCC - SMD/SMT WCAP-CSGP 0.1uF 0805 10% 25V MLCC " H 3800 4875 50  0001 C CNN "Description"
+F 5 "Wurth Elektronik " H 3800 4875 50  0001 C CNN "MFN"
+F 6 "885012207072" H 3800 4875 50  0001 C CNN "MFP"
+F 7 "https://www.mouser.com/ProductDetail/Wurth-Elektronik/885012207072?qs=0KOYDY2FL28rQMV4504TxA%3D%3D" H 3800 4875 50  0001 C CNN "S1PL"
+F 8 "710-885012207072 " H 3800 4875 50  0001 C CNN "S1PN"
 	1    3800 4875
 	1    0    0    -1
@@
 P 4125 4875
 F 0 "C27" H 4250 4925 50  0000 L CNN
-F 1 "10uF" H 4150 4775 50  0000 L CNN
+F 1 "10u" H 4150 4775 50  0000 L CNN
 F 2 "Capacitor_SMD:C_0805_2012Metric_Pad1.15x1.40mm_HandSolder" H 4163 4725 50  0001 C CNN
-F 3 "~" H 4125 4875 50  0001 C CNN
+F 3 "https://www.mouser.com/datasheet/2/585/MLCC-1837944.pdf" H 4125 4875 50  0001 C CNN
+F 4 "Multilayer Ceramic Capacitors MLCC - SMD/SMT 16V 10uF X5R 0805 10%" H 4125 4875 50  0001 C CNN "Description"
+F 5 "Samsung Electro-Mechanics " H 4125 4875 50  0001 C CNN "MFN"
+F 6 "CL21A106KOQNNNG " H 4125 4875 50  0001 C CNN "MFP"
+F 7 "https://www.mouser.com/ProductDetail/Samsung-Electro-Mechanics/CL21A106KOQNNNG?qs=hqM3L16%252BxlcMWI7QbqH0LA%3D%3D" H 4125 4875 50  0001 C CNN "S1PL"
+F 8 " 187-CL21A106KOQNNNG " H 4125 4875 50  0001 C CNN "S1PN"
 	1    4125 4875
 	1    0    0    -1
@@
 P 4825 3450
 F 0 "C28" H 4875 3525 50  0000 L CNN
-F 1 "100nF" H 4850 3350 50  0000 L CNN
+F 1 "100n" H 4850 3350 50  0000 L CNN
 F 2 "Capacitor_SMD:C_0805_2012Metric_Pad1.15x1.40mm_HandSolder" H 4863 3300 50  0001 C CNN
-F 3 "~" H 4825 3450 50  0001 C CNN
+F 3 "https://www.mouser.com/datasheet/2/445/885012207072-1727745.pdf" H 4825 3450 50  0001 C CNN
+F 4 "Multilayer Ceramic Capacitors MLCC - SMD/SMT WCAP-CSGP 0.1uF 0805 10% 25V MLCC " H 4825 3450 50  0001 C CNN "Description"
+F 5 "Wurth Elektronik " H 4825 3450 50  0001 C CNN "MFN"
+F 6 "885012207072" H 4825 3450 50  0001 C CNN "MFP"
+F 7 "https://www.mouser.com/ProductDetail/Wurth-Elektronik/885012207072?qs=0KOYDY2FL28rQMV4504TxA%3D%3D" H 4825 3450 50  0001 C CNN "S1PL"
+F 8 "710-885012207072 " H 4825 3450 50  0001 C CNN "S1PN"
 	1    4825 3450
 	1    0    0    -1
@@
 P 5150 3450
 F 0 "C29" H 5200 3525 50  0000 L CNN
-F 1 "10uF" H 5175 3350 50  0000 L CNN
+F 1 "10u" H 5175 3350 50  0000 L CNN
 F 2 "Capacitor_SMD:C_0805_2012Metric_Pad1.15x1.40mm_HandSolder" H 5188 3300 50  0001 C CNN
-F 3 "~" H 5150 3450 50  0001 C CNN
+F 3 "https://www.mouser.com/datasheet/2/585/MLCC-1837944.pdf" H 5150 3450 50  0001 C CNN
+F 4 "Multilayer Ceramic Capacitors MLCC - SMD/SMT 16V 10uF X5R 0805 10%" H 5150 3450 50  0001 C CNN "Description"
+F 5 "Samsung Electro-Mechanics " H 5150 3450 50  0001 C CNN "MFN"
+F 6 "CL21A106KOQNNNG " H 5150 3450 50  0001 C CNN "MFP"
+F 7 "https://www.mouser.com/ProductDetail/Samsung-Electro-Mechanics/CL21A106KOQNNNG?qs=hqM3L16%252BxlcMWI7QbqH0LA%3D%3D" H 5150 3450 50  0001 C CNN "S1PL"
+F 8 " 187-CL21A106KOQNNNG " H 5150 3450 50  0001 C CNN "S1PN"
 	1    5150 3450
 	1    0    0    -1
@@
 P 5800 3800
 F 0 "C30" V 5950 3700 50  0000 L CNN
-F 1 "100nF" V 5675 3675 50  0000 L CNN
+F 1 "100n" V 5675 3675 50  0000 L CNN
 F 2 "Capacitor_SMD:C_0805_2012Metric_Pad1.15x1.40mm_HandSolder" H 5838 3650 50  0001 C CNN
-F 3 "~" H 5800 3800 50  0001 C CNN
+F 3 "https://www.mouser.com/datasheet/2/445/885012207072-1727745.pdf" H 5800 3800 50  0001 C CNN
+F 4 "Multilayer Ceramic Capacitors MLCC - SMD/SMT WCAP-CSGP 0.1uF 0805 10% 25V MLCC " H 5800 3800 50  0001 C CNN "Description"
+F 5 "Wurth Elektronik " H 5800 3800 50  0001 C CNN "MFN"
+F 6 "885012207072" H 5800 3800 50  0001 C CNN "MFP"
+F 7 "https://www.mouser.com/ProductDetail/Wurth-Elektronik/885012207072?qs=0KOYDY2FL28rQMV4504TxA%3D%3D" H 5800 3800 50  0001 C CNN "S1PL"
+F 8 "710-885012207072 " H 5800 3800 50  0001 C CNN "S1PN"
 	1    5800 3800
 	0    -1   -1   0

Commit message: Updated: New version for board
Parts:
- removed C30: 100n, Capacitor_SMD:C_0805_2012Metric_Pad1.15x1.40mm_HandSolder, symbol Device:C
Connections:
- no-connect marks 2 -> 3
Changed lines of the file:
@@
 Wire Wire Line
 	5500 3400 5500 3700
-Connection ~ 5600 3700
 Wire Wire Line
 	7475 3200 7325 3200
@@
 DOUT
 NoConn ~ 6025 3000
-Wire Wire Line
-	5600 3800 5650 3800
-$Comp
-L Device:C C30
-U 1 1 5E3C27FC
-P 5800 3800
-F 0 "C30" V 5950 3700 50  0000 L CNN
-F 1 "100n" V 5675 3675 50  0000 L CNN
-F 2 "Capacitor_SMD:C_0805_2012Metric_Pad1.15x1.40mm_HandSolder" H 5838 3650 50  0001 C CNN
-F 3 "https://www.mouser.com/datasheet/2/445/885012207072-1727745.pdf" H 5800 3800 50  0001 C CNN
-F 4 "Multilayer Ceramic Capacitors MLCC - SMD/SMT WCAP-CSGP 0.1uF 0805 10% 25V MLCC " H 5800 3800 50  0001 C CNN "Description"
-F 5 "Wurth Elektronik " H 5800 3800 50  0001 C CNN "MFN"
-F 6 "885012207072" H 5800 3800 50  0001 C CNN "MFP"
-F 7 "https://www.mouser.com/ProductDetail/Wurth-Elektronik/885012207072?qs=0KOYDY2FL28rQMV4504TxA%3D%3D" H 5800 3800 50  0001 C CNN "S1PL"
-F 8 "710-885012207072 " H 5800 3800 50  0001 C CNN "S1PN"
-	1    5800 3800
-	0    -1   -1   0
-$EndComp
-Wire Wire Line
-	5600 3700 5600 3800
 Connection ~ 5500 3700
 Wire Wire Line
@@
 	5950 2800 5950 2650
 Wire Wire Line
-	5950 3800 6025 3800
-Wire Wire Line
 	5150 3200 6025 3200
 Wire Wire Line
@@
 Wire Wire Line
 	7325 4200 7475 4200
+NoConn ~ 6025 3800
 $EndSCHEMATC

Commit message: perf: Replace folder libraries to lib_deps in platformio.ini. Previous performance: RAM:   [====      ]  39.1% (used 1001 bytes from 2560 bytes) Flash: [====      ]  40.2% (used 11518 bytes from 28672 bytes)
Current performance:
RAM:   [==        ]  23.5% (used 601 bytes from 2560 bytes)
Flash: [==        ]  22.5% (used 6460 bytes from 28672 bytes)
Changed lines of the file:
@@
 P 3550 4900
 F 0 "SJ1" H 3650 5025 59  0000 R CNN
-F 1 "JUMPER-PAD-2-NC_BY_TRACE" H 4375 5150 59  0000 R CNN
+F 1 "JUMPER-PAD-2-NC_BY_TRACE" H 4250 5200 59  0000 R CNN
 F 2 "Jumper:SolderJumper-2_P1.3mm_Open_RoundedPad1.0x1.5mm" H 3550 4900 50  0001 C CNN
 F 3 "" H 3550 4900 50  0001 C CNN
@@
 Text HLabel 3950 4550 1    59   Input ~ 0
 3.3V
-Text Label 4825 3825 2    59   ~ 0
-LGND
 Wire Wire Line
 	4825 3700 4825 3825
-Text Label 3550 4600 0    59   ~ 0
-LGND
 Text Notes 7100 7000 0    315  ~ 0
 24bits HX711
@@
 Wire Wire Line
 	5600 3600 5600 3700
-Text Label 5650 4000 2    50   ~ 0
-LGND
 Wire Wire Line
 	5650 4000 6025 4000
@@
 	7325 4200 7475 4200
 NoConn ~ 6025 3800
+Text GLabel 5650 4000 0    50   Input ~ 0
+LGND
+Text GLabel 4825 3825 0    50   Input ~ 0
+LGND
+Text GLabel 3550 4600 0    50   Input ~ 0
+LGND
 $EndSCHEMATC

Commit message: refactor: Kicad design
Connections:
- net LGND: no longer U6.7 (INA-)
- net A+: no longer names the net of U6.8 (INA+)
- no-connect marks 3 -> 5
Changed lines of the file:
@@
 	7475 3200 7325 3200
 NoConn ~ 7325 3400
-Wire Wire Line
-	5925 4200 6025 4200
-Text HLabel 5925 4200 0    50   Input ~ 0
-A+
 $Comp
 L Device:R R41
@@
 	5600 3600 5600 3700
 Wire Wire Line
-	5650 4000 6025 4000
-Wire Wire Line
 	5500 3400 6025 3400
 Wire Wire Line
@@
 	7325 4200 7475 4200
 NoConn ~ 6025 3800
-Text GLabel 5650 4000 0    50   Input ~ 0
-LGND
 Text GLabel 4825 3825 0    50   Input ~ 0
 LGND
 Text GLabel 3550 4600 0    50   Input ~ 0
 LGND
+NoConn ~ 6025 4000
+NoConn ~ 6025 4200
 $EndSCHEMATC
