File: pcb/main/Conductometer_2.kicad_sch (KiCad schematic)
At the start: 30 parts, among them J2 Conn_Coaxial_Power, U10 LM2660M, U2 TLV6004PW, U8 CD4060BM

Commit message: feat: update sch
Schematic updated with new BOM
Parts:
- R10, R12, R5, R7, R8, R9: MFN (none) -> KOA Speer; MFP (none) -> RK73H2ATTD3602F; S1PL (none) -> https://www.mouser.com/ProductDetail/KOA-Speer/RK73H2ATTD36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; S1PN (none) -> 660-RK73H2ATTD3602F
- R17: MFN (none) -> YAGEO; MFP (none) -> RC0805FR-0751KL; S1PL (none) -> https://www.mouser.com/ProductDetail/YAGEO/RC0805FR-0751KL?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; S1PN (none) -> 603-RC0805FR-0751KL
- U10: MFN (none) -> Texas Instruments; MFP (none) -> LM2660MX/NOPB; S1PL (none) -> https://www.mouser.com/ProductDetail/Texas-Instruments/LM26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; S1PN (none) -> 926-LM2660MX/NOPB
Changed lines of the file:
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@@
       (effects (font (size 1.27 1.27)) hide)
     )
-    (property "Datasheet" "~" (id 3) (at 146.685 137.795 0)
+    (property "Datasheet" "https://www.mouser.com/datasheet/2/447/Yageo_03_18_2021_PYu_RC_Group_51_RoHS_L_11-2199992.pdf" (id 3) (at 146.685 137.795 0)
+      (effects (font (size 1.27 1.27)) hide)
+    )
+    (property "Description" "Resistores de película gruesa - SMD 51 kOhms 125 mW 0805 1% " (id 4) (at 146.685 137.795 0)
+      (effects (font (size 1.27 1.27)) hide)
+    )
+    (property "MFN" "YAGEO " (id 5) (at 146.685 137.795 0)
+      (effects (font (size 1.27 1.27)) hide)
+    )
+    (property "MFP" "RC0805FR-0751KL " (id 6) (at 146.685 137.795 0)
+      (effects (font (size 1.27 1.27)) hide)
+    )
+    (property "S1PL" "https://www.mouser.com/ProductDetail/YAGEO/RC0805FR-0751KL?qs=sGAEpiMZZMtlubZbdhIBIEM5%252BYIsBt7JhZdNC0q5e2g%3D" (id 7) (at 146.685 137.795 0)
+      (effects (font (size 1.27 1.27)) hide)
+    )
+    (property "S1PN" "603-RC0805FR-0751KL " (id 8) (at 146.685 137.795 0)
       (effects (font (size 1.27 1.27)) hide)
     )
@@
       (effects (font (size 1.524 1.524)) hide)
     )
-    (property "Datasheet" "" (id 3) (at 194.945 32.385 0)
+    (property "Datasheet" "https://www.ti.com/lit/ds/symlink/lm2660.pdf?HQS=dis-mous-null-mousermode-dsf-pf-null-wwe&ts=1653317307356&ref_url=https%253A%252F%252Fwww.mouser.com%252F" (id 3) (at 194.945 32.385 0)
       (effects (font (size 1.524 1.524)))
+    )
+    (property "Description" "Reguladores de voltaje de conmutación Switched Capacitor Vtg Cnvtr " (id 4) (at 194.945 32.385 0)
+      (effects (font (size 1.27 1.27)) hide)
+    )
+    (property "MFN" "Texas Instruments " (id 5) (at 194.945 32.385 0)
+      (effects (font (size 1.27 1.27)) hide)
+    )
+    (property "MFP" "LM2660MX/NOPB " (id 6) (at 194.945 32.385 0)
+      (effects (font (size 1.27 1.27)) hide)
+    )
+    (property "S1PL" "https://www.mouser.com/ProductDetail/Texas-Instruments/LM2660MX-NOPB?qs=X1J7HmVL2ZE03q2omjVTIg%3D%3D" (id 7) (at 194.945 32.385 0)
+      (effects (font (size 1.27 1.27)) hide)
+    )
+    (property "S1PN" "926-LM2660MX/NOPB " (id 8) (at 194.945 32.385 0)
+      (effects (font (size 1.27 1.27)) hide)
     )
     (pin "1")
@@
       (effects (font (size 1.27 1.27)) hide)
     )
-    (property "Datasheet" "~" (id 3) (at 68.58 73.025 0)
+    (property "Datasheet" "https://www.mouser.com/datasheet/2/219/RK73H-1825326.pdf" (id 3) (at 68.58 73.025 0)
+      (effects (font (size 1.27 1.27)) hide)
+    )
+    (property "Description" "Resistores de película gruesa - SMD 1/4W 36K OHM 1% " (id 4) (at 68.58 73.025 0)
+      (effects (font (size 1.27 1.27)) hide)
+    )
+    (property "MFN" "KOA Speer " (id 5) (at 68.58 73.025 0)
+      (effects (font (size 1.27 1.27)) hide)
+    )
+    (property "MFP" "RK73H2ATTD3602F " (id 6) (at 68.58 73.025 0)
+      (effects (font (size 1.27 1.27)) hide)
+    )
+    (property "S1PL" "https://www.mouser.com/ProductDetail/KOA-Speer/RK73H2ATTD3602F?qs=sGAEpiMZZMtlubZbdhIBIGHDdrtfndCCjYVgzAybnVs%3D" (id 7) (at 68.58 73.025 0)
+      (effects (font (size 1.27 1.27)) hide)
+    )
+    (property "S1PN" "660-RK73H2ATTD3602F " (id 8) (at 68.58 73.025 0)
       (effects (font (size 1.27 1.27)) hide)
     )
@@
       (effects (font (size 1.27 1.27)) hide)
     )
-    (property "Datasheet" "~" (id 3) (at 91.44 82.55 0)
+    (property "Datasheet" "https://www.mouser.com/datasheet/2/219/RK73H-1825326.pdf" (id 3) (at 91.44 82.55 0)
+      (effects (font (size 1.27 1.27)) hide)
+    )
+    (property "Description" "Resistores de película gruesa - SMD 1/4W 36K OHM 1% " (id 4) (at 91.44 82.55 0)
+      (effects (font (size 1.27 1.27)) hide)
+    )
+    (property "MFN" "KOA Speer " (id 5) (at 91.44 82.55 0)
+      (effects (font (size 1.27 1.27)) hide)
+    )
+    (property "MFP" "RK73H2ATTD3602F " (id 6) (at 91.44 82.55 0)
+      (effects (font (size 1.27 1.27)) hide)
+    )
+    (property "S1PL" "https://www.mouser.com/ProductDetail/KOA-Speer/RK73H2ATTD3602F?qs=sGAEpiMZZMtlubZbdhIBIGHDdrtfndCCjYVgzAybnVs%3D" (id 7) (at 91.44 82.55 0)
+      (effects (font (size 1.27 1.27)) hide)
+    )
+    (property "S1PN" "660-RK73H2ATTD3602F " (id 8) (at 91.44 82.55 0)
       (effects (font (size 1.27 1.27)) hide)
     )
@@
       (effects (font (size 1.27 1.27)) hide)
     )
-    (property "Datasheet" "~" (id 3) (at 85.09 55.88 0)
+    (property "Datasheet" "https://www.mouser.com/datasheet/2/219/RK73H-1825326.pdf" (id 3) (at 85.09 55.88 0)
+      (effects (font (size 1.27 1.27)) hide)
+    )
+    (property "Description" "Resistores de película gruesa - SMD 1/4W 36K OHM 1% " (id 4) (at 85.09 55.88 0)
+      (effects (font (size 1.27 1.27)) hide)
+    )
+    (property "MFN" "KOA Speer " (id 5) (at 85.09 55.88 0)
+      (effects (font (size 1.27 1.27)) hide)
+    )
+    (property "MFP" "RK73H2ATTD3602F " (id 6) (at 85.09 55.88 0)
+      (effects (font (size 1.27 1.27)) hide)
+    )
+    (property "S1PL" "https://www.mouser.com/ProductDetail/KOA-Speer/RK73H2ATTD3602F?qs=sGAEpiMZZMtlubZbdhIBIGHDdrtfndCCjYVgzAybnVs%3D" (id 7) (at 85.09 55.88 0)
+      (effects (font (size 1.27 1.27)) hide)
+    )
+    (property "S1PN" "660-RK73H2ATTD3602F " (id 8) (at 85.09 55.88 0)
       (effects (font (size 1.27 1.27)) hide)
     )
@@
       (effects (font (size 1.27 1.27)) hide)
     )
-    (property "Datasheet" "~" (id 3) (at 104.14 55.88 0)
+    (property "Datasheet" "https://www.mouser.com/datasheet/2/219/RK73H-1825326.pdf" (id 3) (at 104.14 55.88 0)
+      (effects (font (size 1.27 1.27)) hide)
+    )
+    (property "Description" "Resistores de película gruesa - SMD 1/4W 36K OHM 1% " (id 4) (at 104.14 55.88 0)
+      (effects (font (size 1.27 1.27)) hide)
+    )
+    (property "MFN" "KOA Speer " (id 5) (at 104.14 55.88 0)
+      (effects (font (size 1.27 1.27)) hide)
+    )
+    (property "MFP" "RK73H2ATTD3602F " (id 6) (at 104.14 55.88 0)
+      (effects (font (size 1.27 1.27)) hide)
+    )
+    (property "S1PL" "https://www.mouser.com/ProductDetail/KOA-Speer/RK73H2ATTD3602F?qs=sGAEpiMZZMtlubZbdhIBIGHDdrtfndCCjYVgzAybnVs%3D" (id 7) (at 104.14 55.88 0)
+      (effects (font (size 1.27 1.27)) hide)
+    )
+    (property "S1PN" "660-RK73H2ATTD3602F " (id 8) (at 104.14 55.88 0)
       (effects (font (size 1.27 1.27)) hide)
     )
@@
       (effects (font (size 1.27 1.27)) hide)
     )
-    (property "Datasheet" "~" (id 3) (at 116.84 55.88 0)
+    (property "Datasheet" "https://www.mouser.com/datasheet/2/219/RK73H-1825326.pdf" (id 3) (at 116.84 55.88 0)
+      (effects (font (size 1.27 1.27)) hide)
+    )
+    (property "Description" "Resistores de película gruesa - SMD 1/4W 36K OHM 1% " (id 4) (at 116.84 55.88 0)
+      (effects (font (size 1.27 1.27)) hide)
+    )
+    (property "MFN" "KOA Speer " (id 5) (at 116.84 55.88 0)
+      (effects (font (size 1.27 1.27)) hide)
+    )
+    (property "MFP" "RK73H2ATTD3602F " (id 6) (at 116.84 55.88 0)
+      (effects (font (size 1.27 1.27)) hide)
+    )
+    (property "S1PL" "https://www.mouser.com/ProductDetail/KOA-Speer/RK73H2ATTD3602F?qs=sGAEpiMZZMtlubZbdhIBIGHDdrtfndCCjYVgzAybnVs%3D" (id 7) (at 116.84 55.88 0)
+      (effects (font (size 1.27 1.27)) hide)
+    )
+    (property "S1PN" "660-RK73H2ATTD3602F " (id 8) (at 116.84 55.88 0)
       (effects (font (size 1.27 1.27)) hide)
     )
@@
       (effects (font (size 1.27 1.27)) hide)
     )
-    (property "Datasheet" "~" (id 3) (at 137.16 67.945 0)
-      (effects (font (size 1.27 1.27)) hide)
-    )
+    (property "Datasheet" "https://www.mouser.com/datasheet/2/219/RK73H-1825326.pdf" (id 3) (at 137.16 67.945 0)
+      (effects (font (size 1.27 1.27)) hide)
+    )
+    (property "Description" "Resistores de película gruesa - SMD 1/4W 36K OHM 1% " (id 4) (at 137.16 67.945 0)
+      (effects (font (size 1.27 1.27)) hide)
+    )
+    (property "MFN" "KOA Speer " (id 5) (at 137.16 67.945 0)
+      (effects (font (size 1.27 1.27)) hide)
+    )
+    (property "MFP" "RK73H2ATTD3602F " (id 6) (at 137.16 67.945 0)
+      (effects (font (size 1.27 1.27)) hide)
+    )
+    (property "S1PL" "https://www.mouser.com/ProductDetail/KOA-Speer/RK73H2ATTD3602F?qs=sGAEpiMZZMtlubZbdhIBIGHDdrtfndCCjYVgzAybnVs%3D" (id 7) (at 137.16 67.945 0)
+      (effects (font (size 1.27 1.27)) hide)
+    )
+    (property "S1PN" "660-RK73H2ATTD3602F " (id 8) (at 137.16 67.945 0)
+      (effects (font (size 1.27 1.27)) hide)
+    )

Commit message: feat: new PCB version to 1.1.2
Schematic:
- Updated sheets to 1.1.2 version.
- Change inputs for last OPA in EC sheet.
- INA- and INA+ set to GND in 24bits sheet for reduce noise.
- Change /CE connection (TX -> HWB) in Memory and COMM LED.
- Adding a correct guard in pH sheet.
- Adding correct 12 V support for 3.3 V (avoid battery charge circuit).

Design:
- Increase width track for 2 A in 3.3 V power supply.
- Order labels.
- Put new schottky diode for 12 V -> 3.3 V circuit direct connection.
- Adding pH and EC tag.
- Adding guard and restrict area for pH adquisiton.
Parts:
- C35: value 20p -> 220n
- R12: value 36k -> 10k
Connections:
- net at R10.2, R9.1: now also U2.13 (-); no longer U2.12 (+)
- net at D2.1 (K), R8.1: now also U2.12 (+); no longer U2.13 (-)
- net CT1 renamed ECINPUT
- net CT2 renamed ECOUTPUT
Other:
- company: (none) -> Hackuarium
- title: (none) -> EC adquisition
Changed lines of the file:
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@@
   (paper "A4")
   (title_block
-    (date "2021-11-26")
-    (rev "0.1")
+    (title "EC adquisition")
+    (date "2022-07-25")
+    (rev "1.1.2")
+    (company "Hackuarium")
   )
   (junction (at 143.51 67.945) (diameter 0) (color 0 0 0 0)
@@
     (stroke (width 0) (type default) (color 0 0 0 0))
   )
-  (global_label "CT2" (shape input) (at 33.655 75.565 180) (fields_autoplaced)
+  (global_label "ECOUTPUT" (shape input) (at 33.655 75.565 180) (fields_autoplaced)
     (effects (font (size 1.27 1.27)) (justify right))
-    (property "Intersheet References" "${INTERSHEET_REFS}" (id 0) (at 0 0 0)
-      (effects (font (size 1.27 1.27)) hide)
-    )
-  )
-  (global_label "CT1" (shape input) (at 250.19 120.65 90) (fields_autoplaced)
+    (property "Intersheet References" "${INTERSHEET_REFS}" (id 0) (at 21.4357 75.4856 0)
+      (effects (font (size 1.27 1.27)) (justify right) hide)
+    )
+  )
+  (global_label "ECINPUT" (shape input) (at 250.19 120.65 90) (fields_autoplaced)
     (effects (font (size 1.27 1.27)) (justify left))
-    (property "Intersheet References" "${INTERSHEET_REFS}" (id 0) (at 0 0 0)
-      (effects (font (size 1.27 1.27)) hide)
-    )
-  )
-  (global_label "CT1" (shape input) (at 175.26 140.335 0) (fields_autoplaced)
+    (property "Intersheet References" "${INTERSHEET_REFS}" (id 0) (at 250.1106 110.124 90)
+      (effects (font (size 1.27 1.27)) (justify left) hide)
+    )
+  )
+  (global_label "ECINPUT" (shape input) (at 175.26 140.335 0) (fields_autoplaced)
     (effects (font (size 1.27 1.27)) (justify left))
-    (property "Intersheet References" "${INTERSHEET_REFS}" (id 0) (at 0 0 0)
-      (effects (font (size 1.27 1.27)) hide)
-    )
-  )
-  (global_label "CT2" (shape input) (at 250.19 133.35 270) (fields_autoplaced)
+    (property "Intersheet References" "${INTERSHEET_REFS}" (id 0) (at 185.786 140.2556 0)
+      (effects (font (size 1.27 1.27)) (justify left) hide)
+    )
+  )
+  (global_label "ECOUTPUT" (shape input) (at 250.19 133.35 270) (fields_autoplaced)
     (effects (font (size 1.27 1.27)) (justify right))
-    (property "Intersheet References" "${INTERSHEET_REFS}" (id 0) (at 0 0 0)
-      (effects (font (size 1.27 1.27)) hide)
+    (property "Intersheet References" "${INTERSHEET_REFS}" (id 0) (at 250.1106 145.5693 90)
+      (effects (font (size 1.27 1.27)) (justify right) hide)
     )
   )
@@
     (pin "2")
   )
-  (symbol (lib_id "bioreactor:TLV6004PW") (at 120.65 67.945 0) (unit 4)
-    (in_bom yes) (on_board yes)
-    (property "Reference" "U2" (id 0) (at 120.65 58.6232 0))
-    (property "Value" "TLV6004PW" (id 1) (at 120.65 60.9346 0))
-    (property "Footprint" "Package_SO:TSSOP-14_4.4x5mm_P0.65mm" (id 2) (at 121.92 78.105 0)
-      (effects (font (size 1.27 1.27)) hide)
-    )
-    (property "Datasheet" "https://www.ti.com/lit/ds/symlink/tlv6004.pdf?ts=1591554967798&ref_url=https://www.ti.com/product/TLV6004" (id 3) (at 121.92 62.865 0)
+  (symbol (lib_id "bioreactor:TLV6004PW") (at 120.65 67.945 0) (mirror x) (unit 4)
+    (in_bom yes) (on_board yes)
+    (property "Reference" "U2" (id 0) (at 120.65 77.2668 0))
+    (property "Value" "TLV6004PW" (id 1) (at 120.65 74.9554 0))
+    (property "Footprint" "Package_SO:TSSOP-14_4.4x5mm_P0.65mm" (id 2) (at 121.92 57.785 0)
+      (effects (font (size 1.27 1.27)) hide)
+    )
+    (property "Datasheet" "https://www.ti.com/lit/ds/symlink/tlv6004.pdf?ts=1591554967798&ref_url=https://www.ti.com/product/TLV6004" (id 3) (at 121.92 73.025 0)
       (effects (font (size 1.27 1.27)) hide)
     )
@@
     (in_bom yes) (on_board yes)
     (property "Reference" "R12" (id 0) (at 137.16 62.6872 90))
-    (property "Value" "36k" (id 1) (at 137.16 64.9986 90))
+    (property "Value" "10k" (id 1) (at 137.16 64.9986 90))
     (property "Footprint" "Resistor_SMD:R_0805_2012Metric_Pad1.20x1.40mm_HandSolder" (id 2) (at 137.16 66.167 90)
       (effects (font (size 1.27 1.27)) hide)
@@
       (effects (font (size 1.27 1.27)) (justify left))
     )
-    (property "Value" "20p" (id 1) (at 146.431 75.438 0)
-      (effects (font (size 1.27 1.27)) (justify left))
-    )
+    (property "Value" "220n" (id 1) (at 146.431 75.438 0)
+      (effects (font (size 1.27 1.27)) (justify left))
+    )

Commit message: test: version 1.1.2
Some bugs are into semphore (ADC or memory access).
Parts:
- U10: value LM2660M -> (none); footprint pHMeter:LM2660M -> (none)
- U8: value CD4060BM -> (none)
Changed lines of the file:
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@@
     (pin "2")
     (pin "3")
+    (pin "5")
+    (pin "6")
+    (pin "7")
+    (pin "10")
+    (pin "8")
+    (pin "9")
+    (pin "12")
+    (pin "13")
+    (pin "14")
+    (pin "11")
+    (pin "4")
   )
   (symbol (lib_id "bioreactor:TLV6004PW") (at 52.07 73.025 0) (unit 2)
@@
       (effects (font (size 1.27 1.27)) hide)
     )
+    (pin "1")
+    (pin "2")
+    (pin "3")
     (pin "5")
     (pin "6")
     (pin "7")
+    (pin "10")
+    (pin "8")
+    (pin "9")
+    (pin "12")
+    (pin "13")
+    (pin "14")
+    (pin "11")
+    (pin "4")
   )
   (symbol (lib_id "bioreactor:TLV6004PW") (at 88.265 70.485 0) (unit 3)
@@
       (effects (font (size 1.27 1.27)) hide)
     )
+    (pin "1")
+    (pin "2")
+    (pin "3")
+    (pin "5")
+    (pin "6")
+    (pin "7")
     (pin "10")
     (pin "8")
     (pin "9")
-  )
-  (symbol (lib_id "bioreactor:TLV6004PW") (at 86.36 22.225 90) (unit 5)
-    (in_bom yes) (on_board yes)
-    (property "Reference" "U2" (id 0) (at 85.1916 23.2918 0)
-      (effects (font (size 1.27 1.27)) (justify left))
-    )
-    (property "Value" "TLV6004PW" (id 1) (at 87.503 23.2918 0)
-      (effects (font (size 1.27 1.27)) (justify left))
-    )
-    (property "Footprint" "Package_SO:TSSOP-14_4.4x5mm_P0.65mm" (id 2) (at 96.52 20.955 0)
-      (effects (font (size 1.27 1.27)) hide)
-    )
-    (property "Datasheet" "https://www.ti.com/lit/ds/symlink/tlv6004.pdf?ts=1591554967798&ref_url=https://www.ti.com/product/TLV6004" (id 3) (at 81.28 20.955 0)
-      (effects (font (size 1.27 1.27)) hide)
-    )
+    (pin "12")
+    (pin "13")
+    (pin "14")
     (pin "11")
     (pin "4")
   )
+  (symbol (lib_id "bioreactor:TLV6004PW") (at 86.36 22.225 90) (unit 5)
+    (in_bom yes) (on_board yes)
+    (property "Reference" "U2" (id 0) (at 85.1916 23.2918 0)
+      (effects (font (size 1.27 1.27)) (justify left))
+    )
+    (property "Value" "TLV6004PW" (id 1) (at 87.503 23.2918 0)
+      (effects (font (size 1.27 1.27)) (justify left))
+    )
+    (property "Footprint" "Package_SO:TSSOP-14_4.4x5mm_P0.65mm" (id 2) (at 96.52 20.955 0)
+      (effects (font (size 1.27 1.27)) hide)
+    )
+    (property "Datasheet" "https://www.ti.com/lit/ds/symlink/tlv6004.pdf?ts=1591554967798&ref_url=https://www.ti.com/product/TLV6004" (id 3) (at 81.28 20.955 0)
+      (effects (font (size 1.27 1.27)) hide)
+    )
+    (pin "1")
+    (pin "2")
+    (pin "3")
+    (pin "5")
+    (pin "6")
+    (pin "7")
+    (pin "10")
+    (pin "8")
+    (pin "9")
+    (pin "12")
+    (pin "13")
+    (pin "14")
+    (pin "11")
+    (pin "4")
+  )
   (symbol (lib_id "pHMeter-rescue:CD4060BM-CD4060BM") (at 137.795 122.555 0) (mirror y) (unit 1)
     (in_bom yes) (on_board yes)
@@
       (effects (font (size 1.524 1.524)))
     )
-    (property "Value" "CD4060BM" (id 1) (at 107.315 115.4176 0)
+    (property "Value" "" (id 1) (at 107.315 115.4176 0)
       (effects (font (size 1.524 1.524)))
     )
@@
     )
     (property "Datasheet" "https://www.ti.com/lit/ds/symlink/cd4060b.pdf?ts=1650867032555" (id 3) (at 137.795 122.555 0)
-      (effects (font (size 1.524 1.524)))
+      (effects (font (size 1.524 1.524)) hide)
     )
     (pin "1")
@@
       (effects (font (size 1.524 1.524)))
     )
-    (property "Value" "LM2660M" (id 1) (at 222.885 25.2476 0)
+    (property "Value" "" (id 1) (at 222.885 25.2476 0)
       (effects (font (size 1.524 1.524)))
     )
-    (property "Footprint" "pHMeter:LM2660M" (id 2) (at 222.885 26.289 0)
+    (property "Footprint" "" (id 2) (at 222.885 26.289 0)
       (effects (font (size 1.524 1.524)) hide)
     )
     (property "Datasheet" "https://www.ti.com/lit/ds/symlink/lm2660.pdf?HQS=dis-mous-null-mousermode-dsf-pf-null-wwe&ts=1653317307356&ref_url=https%253A%252F%252Fwww.mouser.com%252F" (id 3) (at 194.945 32.385 0)
-      (effects (font (size 1.524 1.524)))
+      (effects (font (size 1.524 1.524)) hide)
     )
     (property "Description" "Reguladores de voltaje de conmutación Switched Capacitor Vtg Cnvtr " (id 4) (at 194.945 32.385 0)
@@
       (effects (font (size 1.27 1.27)) hide)
     )
+    (pin "1")
+    (pin "2")
+    (pin "3")
+    (pin "5")
+    (pin "6")
+    (pin "7")
+    (pin "10")
+    (pin "8")
+    (pin "9")
     (pin "12")
     (pin "13")
     (pin "14")
+    (pin "11")
+    (pin "4")
   )
   (symbol (lib_id "Bertha_main-eagle-import:GND") (at 75.565 67.945 270) (unit 1)

Commit message: feat: Updated Conductometer sch
Updated descriptions for CD4060
Parts:
- U8: MFN (none) -> Texas Instruments; MFP (none) -> CD4060BNSR; S1PL (none) -> https://www.mouser.com/ProductDetail/Texas-Instruments/CD40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; S1PN (none) -> 595-CD4060BNSR
Changed lines of the file:
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@@
       (effects (font (size 1.524 1.524)) hide)
+    )
+    (property "Description" "CMOS 14-Stage Ripple-Carry Binary Counter/Divider and Oscillator" (id 4) (at 137.795 122.555 0)
+      (effects (font (size 1.27 1.27)) hide)
+    )
+    (property "MFN" "Texas Instruments " (id 5) (at 137.795 122.555 0)
+      (effects (font (size 1.27 1.27)) hide)
+    )
+    (property "MFP" "CD4060BNSR " (id 6) (at 137.795 122.555 0)
+      (effects (font (size 1.27 1.27)) hide)
+    )
+    (property "S1PL" "https://www.mouser.com/ProductDetail/Texas-Instruments/CD4060BNSR?qs=LU5rZWrBGo3rlL%252BliYO71g%3D%3D" (id 7) (at 137.795 122.555 0)
+      (effects (font (size 1.27 1.27)) hide)
+    )
+    (property "S1PN" "595-CD4060BNSR " (id 8) (at 137.795 122.555 0)
+      (effects (font (size 1.27 1.27)) hide)
     )
     (pin "1")

Commit message: feat: updated BOM information
Some components are still without MNF and Seller information
Parts:
- C10, C30, C32, C4: value 10u -> (none); footprint Capacitor_SMD:C_0805_2012Metric_Pad1.18x1.45mm_HandSolder -> (none)
- C12, C2, C34, C8: value 100n -> (none); footprint Capacitor_SMD:C_0805_2012Metric_Pad1.18x1.45mm_HandSolder -> (none)
- C35: value 220n -> (none); footprint Capacitor_SMD:C_0805_2012Metric_Pad1.18x1.45mm_HandSolder -> (none)
- C36, C37: value 100u -> (none); footprint Capacitor_SMD:CP_Elec_8x10 -> (none)
- C5: value 1.5n -> (none); footprint Capacitor_SMD:C_0805_2012Metric_Pad1.18x1.45mm_HandSolder -> (none)
- D1, D2: value 1N4148W -> (none); footprint Diode_SMD:D_SOD-123 -> (none)
- D6: value 1N5819 -> (none); footprint Diode_SMD:D_SOD-123 -> (none)
- J2: value Conn_Coaxial_Power -> (none); footprint Connector_Coaxial:BNC_TEConnectivity_1478204_Vertical -> (none)
- R1: value 820 -> (none); footprint Resistor_SMD:R_0805_2012Metric_Pad1.20x1.40mm_HandSolder -> (none)
- R10, R5, R7, R8, R9: value 36k -> (none); footprint Resistor_SMD:R_0805_2012Metric_Pad1.20x1.40mm_HandSolder -> (none)
- R12, R6: value 10k -> (none); footprint Resistor_SMD:R_0805_2012Metric_Pad1.20x1.40mm_HandSolder -> (none)
- R17: value 51k -> (none); footprint Resistor_SMD:R_0805_2012Metric_Pad1.20x1.40mm_HandSolder -> (none)
- R18: value 2k -> (none); footprint Resistor_SMD:R_0805_2012Metric_Pad1.20x1.40mm_HandSolder -> (none)
- R2: value 100k -> (none); footprint Resistor_SMD:R_0805_2012Metric_Pad1.20x1.40mm_HandSolder -> (none); MFN (none) -> Vishay / Dale; MFP (none) -> CRCW0805100KJNEC; S1PL (none) -> https://www.mouser.com/ProductDetail/Vishay-Dale/CRCW080510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; S1PN (none) -> 71-CRCW0805100KJNEC
- U2: value TLV6004PW -> (none); footprint Package_SO:TSSOP-14_4.4x5mm_P0.65mm -> (none)
