File: pcb/main/Conductometer_2.kicad_sch (KiCad schematic)
At the start: 30 parts

Commit message: feat: updated BOM
Parts:
- C10, C30, C32, C4: value (none) -> 10u; footprint (none) -> Capacitor_SMD:C_0805_2012Metric_Pad1.18x1.45mm_HandSolder
- C12, C2, C34, C8: value (none) -> 100n; footprint (none) -> Capacitor_SMD:C_0805_2012Metric_Pad1.18x1.45mm_HandSolder
- C35: value (none) -> 220n; footprint (none) -> Capacitor_SMD:C_0805_2012Metric_Pad1.18x1.45mm_HandSolder
- C36, C37: value (none) -> 100u; footprint (none) -> Capacitor_SMD:CP_Elec_8x10
- C5: value (none) -> 1.5n
- D1, D2: value (none) -> 1N4148W; footprint (none) -> Diode_SMD:D_SOD-123; MFN (none) -> Panjit; MFP (none) -> 1N4148W_R1_00001; S1PL (none) -> https://www.mouser.com/ProductDetail/Panjit/1N4148W_R1_0000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; S1PN (none) -> 241-1N4148W_R1_00001
- D6: value (none) -> 1N5819
- J2: value (none) -> Conn_Coaxial_Power; footprint (none) -> Connector_Coaxial:BNC_TEConnectivity_1478204_Vertical; MFN (none) -> Amphenol RF; MFP (none) -> 112404; S1PL (none) -> https://www.mouser.com/ProductDetail/Amphenol-RF/112404?qs=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; S1PN (none) -> 523-112404
- R1: value (none) -> 820
- R10, R5, R7, R8, R9: value (none) -> 36k
- R12, R6: value (none) -> 10k
- R17: value (none) -> 51k
- R18: value (none) -> 2k
- R2: value (none) -> 100k
- U10: value (none) -> LM2660M
- U2: value (none) -> TLV6004PW; footprint (none) -> Package_SO:TSSOP-14_4.4x5mm_P0.65mm; MFN (none) -> Texas Instruments; MFP (none) -> TLV6004IPWR; S1PL (none) -> https://www.mouser.com/ProductDetail/Texas-Instruments/TLV6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; S1PN (none) -> 595-TLV6004IPWR
- U8: value (none) -> CD4060BM; footprint (none) -> Package_SO:SOIC-16_3.9x9.9mm_P1.27mm
