File: pcb/main/pH.kicad_sch (KiCad schematic)
At the start: 9 parts

Commit message: feat: updated BOM
Parts:
- C1, C3: value (none) -> 100n; footprint (none) -> Capacitor_SMD:C_0805_2012Metric_Pad1.18x1.45mm_HandSolder
- C9: value (none) -> 22u; footprint (none) -> Capacitor_SMD:C_0805_2012Metric_Pad1.15x1.40mm_HandSolder
- J3: value (none) -> Conn_Coaxial_Power; footprint (none) -> Connector_Coaxial:BNC_TEConnectivity_1478204_Vertical
- R11: value (none) -> 56.2k; footprint (none) -> Resistor_SMD:R_0805_2012Metric_Pad1.15x1.40mm_HandSolder
- R13, R3, R4: value (none) -> 10k; footprint (none) -> Resistor_SMD:R_0805_2012Metric_Pad1.20x1.40mm_HandSolder
- U1: value (none) -> TLV6004PW; footprint (none) -> Package_SO:TSSOP-14_4.4x5mm_P0.65mm; MFN (none) -> Texas Instruments; MFP (none) -> TLV6004IPWR; S1PL (none) -> https://www.mouser.com/ProductDetail/Texas-Instruments/TLV6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; S1PN (none) -> 595-TLV6004IPWR
