File: pcb/main/24bits ADC.kicad_sch (KiCad schematic)
At the start: 8 parts, among them J8 SJ, U6 HX711

Commit message: feat: new PCB version to 1.1.2
Schematic:
- Updated sheets to 1.1.2 version.
- Change inputs for last OPA in EC sheet.
- INA- and INA+ set to GND in 24bits sheet for reduce noise.
- Change /CE connection (TX -> HWB) in Memory and COMM LED.
- Adding a correct guard in pH sheet.
- Adding correct 12 V support for 3.3 V (avoid battery charge circuit).

Design:
- Increase width track for 2 A in 3.3 V power supply.
- Order labels.
- Put new schottky diode for 12 V -> 3.3 V circuit direct connection.
- Adding pH and EC tag.
- Adding guard and restrict area for pH adquisiton.
Connections:
- net LGND: now also U6.7 (INA-), U6.8 (INA+)
- no-connect marks 5 -> 3
Other:
- note added: "Default RATE: Closed - Data rate set to 10SPS Open jumper to set to 80SPS Increases noise per read"
- note removed: "24bits HX711"
- note removed: "Default: Closed - Data rate set to 10SPS Open jumper to set to 80SPS Increases noise per read"
- company: (none) -> Hackuarium
- title: (none) -> pH Adquisition
Changed lines of the file:
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@@
 (kicad_sch (version 20211123) (generator eeschema)
   (paper "A4")
+  (title_block
+    (title "pH Adquisition")
+    (date "2022-07-25")
+    (rev "1.1.2")
+    (company "Hackuarium")
+    (comment 1 "pH reading with HX711 24 bits ADC")
+  )
   (junction (at 130.81 93.98) (diameter 0) (color 0 0 0 0)
   )
@@
   (junction (at 122.555 81.28) (diameter 0) (color 0 0 0 0)
   )
+  (junction (at 151.13 106.68) (diameter 0) (color 0 0 0 0)
+  )
   (junction (at 130.81 81.28) (diameter 0) (color 0 0 0 0)
   )
   (junction (at 100.965 129.54) (diameter 0) (color 0 0 0 0)
   )
-  (no_connect (at 153.035 101.6))
-  (no_connect (at 153.035 106.68))
   (no_connect (at 153.035 96.52))
   (no_connect (at 186.055 86.36))
@@
     (stroke (width 0) (type default) (color 0 0 0 0))
   )
+  (wire (pts (xy 151.13 106.68) (xy 151.13 110.49))
+    (stroke (width 0) (type default) (color 0 0 0 0))
+  )
   (wire (pts (xy 104.775 120.015) (xy 104.775 118.745))
     (stroke (width 0) (type default) (color 0 0 0 0))
@@
   )
   (wire (pts (xy 130.81 83.82) (xy 130.81 81.28))
+    (stroke (width 0) (type default) (color 0 0 0 0))
+  )
+  (wire (pts (xy 153.035 101.6) (xy 151.13 101.6))
+    (stroke (width 0) (type default) (color 0 0 0 0))
+  )
+  (wire (pts (xy 151.13 101.6) (xy 151.13 106.68))
     (stroke (width 0) (type default) (color 0 0 0 0))
   )
@@
     (stroke (width 0) (type default) (color 0 0 0 0))
   )
+  (wire (pts (xy 151.13 106.68) (xy 153.035 106.68))
+    (stroke (width 0) (type default) (color 0 0 0 0))
+  )
   (wire (pts (xy 196.215 76.2) (xy 192.405 76.2))
     (stroke (width 0) (type default) (color 0 0 0 0))
@@
     (stroke (width 0) (type default) (color 0 0 0 0))
   )
-  (text "24bits HX711" (at 180.34 177.8 0)
-    (effects (font (size 8.001 8.001)) (justify left bottom))
-  )
-  (text "Default: Closed - Data rate set to 10SPS\n\nOpen jumper to set to 80SPS\nIncreases noise per read"
-    (at 190.5 130.175 0)
+  (text "Default RATE: Closed - Data rate set to 10SPS\n\nOpen jumper to set to 80SPS\nIncreases noise per read"
+    (at 193.04 130.175 0)
     (effects (font (size 1.397 1.397)) (justify right bottom))
   )
@@
       (effects (font (size 1.27 1.27)) hide)
     )
+  )
+  (global_label "LGND" (shape input) (at 151.13 110.49 180) (fields_autoplaced)
+    (effects (font (size 1.27 1.27)) (justify right))
+    (property "Intersheet References" "${INTERSHEET_REFS}" (id 0) (at 28.575 13.335 0)
+      (effects (font (size 1.27 1.27)) hide)
+    )

Commit message: feat: updated BOM information
Some components are still without MNF and Seller information
Parts:
- C26, C28: value 100n -> (none); footprint Capacitor_SMD:C_0805_2012Metric_Pad1.18x1.45mm_HandSolder -> (none)
- C27, C29: value 10u -> (none); footprint Capacitor_SMD:C_0805_2012Metric_Pad1.18x1.45mm_HandSolder -> (none)
- J8: value SJ -> (none); footprint Jumper:SolderJumper-2_P1.3mm_Open_RoundedPad1.0x1.5mm -> (none)
- R41: value 10k -> (none); footprint Resistor_SMD:R_0805_2012Metric_Pad1.20x1.40mm_HandSolder -> (none)
- SJ1: value JUMPER-PAD-2-NC_BY_TRACE -> (none); footprint Jumper:SolderJumper-2_P1.3mm_Open_RoundedPad1.0x1.5mm -> (none)
- U6: value HX711 -> (none); footprint Package_SO:SOIC-16_3.9x9.9mm_P1.27mm -> (none)
Changed lines of the file:
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@@
       (effects (font (size 1.4986 1.4986)) (justify right))
     )
-    (property "Value" "JUMPER-PAD-2-NC_BY_TRACE" (id 1) (at 82.55 106.68 0)
+    (property "Value" "" (id 1) (at 82.55 106.68 0)
       (effects (font (size 1.4986 1.4986)) (justify right))
     )
-    (property "Footprint" "Jumper:SolderJumper-2_P1.3mm_Open_RoundedPad1.0x1.5mm" (id 2) (at 90.17 124.46 0)
+    (property "Footprint" "" (id 2) (at 90.17 124.46 0)
       (effects (font (size 1.27 1.27)) hide)
     )
@@
       (effects (font (size 1.27 1.27)) (justify left))
     )
-    (property "Value" "100n" (id 1) (at 97.155 126.365 0)
+    (property "Value" "" (id 1) (at 97.155 126.365 0)
       (effects (font (size 1.27 1.27)) (justify left))
     )
-    (property "Footprint" "Capacitor_SMD:C_0805_2012Metric_Pad1.18x1.45mm_HandSolder" (id 2) (at 97.4852 127.635 0)
+    (property "Footprint" "" (id 2) (at 97.4852 127.635 0)
       (effects (font (size 1.27 1.27)) hide)
     )
@@
       (effects (font (size 1.27 1.27)) (justify left))
     )
-    (property "Value" "10u" (id 1) (at 105.41 126.365 0)
+    (property "Value" "" (id 1) (at 105.41 126.365 0)
       (effects (font (size 1.27 1.27)) (justify left))
     )
-    (property "Footprint" "Capacitor_SMD:C_0805_2012Metric_Pad1.18x1.45mm_HandSolder" (id 2) (at 105.7402 127.635 0)
+    (property "Footprint" "" (id 2) (at 105.7402 127.635 0)
       (effects (font (size 1.27 1.27)) hide)
     )
@@
       (effects (font (size 1.27 1.27)) (justify left))
     )
-    (property "Value" "100n" (id 1) (at 123.19 90.17 0)
+    (property "Value" "" (id 1) (at 123.19 90.17 0)
       (effects (font (size 1.27 1.27)) (justify left))
     )
-    (property "Footprint" "Capacitor_SMD:C_0805_2012Metric_Pad1.18x1.45mm_HandSolder" (id 2) (at 123.5202 91.44 0)
+    (property "Footprint" "" (id 2) (at 123.5202 91.44 0)
       (effects (font (size 1.27 1.27)) hide)
     )
@@
       (effects (font (size 1.27 1.27)) (justify left))
     )
-    (property "Value" "10u" (id 1) (at 131.445 90.17 0)
+    (property "Value" "" (id 1) (at 131.445 90.17 0)
       (effects (font (size 1.27 1.27)) (justify left))
     )
-    (property "Footprint" "Capacitor_SMD:C_0805_2012Metric_Pad1.18x1.45mm_HandSolder" (id 2) (at 131.7752 91.44 0)
+    (property "Footprint" "" (id 2) (at 131.7752 91.44 0)
       (effects (font (size 1.27 1.27)) hide)
     )
@@
       (effects (font (size 1.4986 1.4986)))
     )
-    (property "Value" "SJ" (id 1) (at 198.755 78.74 0)
+    (property "Value" "" (id 1) (at 198.755 78.74 0)
       (effects (font (size 1.4986 1.4986)))
     )
-    (property "Footprint" "Jumper:SolderJumper-2_P1.3mm_Open_RoundedPad1.0x1.5mm" (id 2) (at 198.755 76.2 0)
+    (property "Footprint" "" (id 2) (at 198.755 76.2 0)
       (effects (font (size 1.27 1.27)) hide)
     )
@@
       (effects (font (size 1.27 1.27)) (justify left))
     )
-    (property "Value" "10k" (id 1) (at 192.405 73.025 90)
+    (property "Value" "" (id 1) (at 192.405 73.025 90)
       (effects (font (size 1.27 1.27)) (justify left))
     )
-    (property "Footprint" "Resistor_SMD:R_0805_2012Metric_Pad1.20x1.40mm_HandSolder" (id 2) (at 190.627 71.12 90)
+    (property "Footprint" "" (id 2) (at 190.627 71.12 90)
       (effects (font (size 1.27 1.27)) hide)
     )
@@
       (effects (font (size 1.4986 1.4986)))
     )
-    (property "Value" "HX711" (id 1) (at 169.545 66.5226 0)
+    (property "Value" "" (id 1) (at 169.545 66.5226 0)
       (effects (font (size 1.4986 1.4986)))
     )
-    (property "Footprint" "Package_SO:SOIC-16_3.9x9.9mm_P1.27mm" (id 2) (at 170.815 115.57 0)
+    (property "Footprint" "" (id 2) (at 170.815 115.57 0)
       (effects (font (size 1.27 1.27)) hide)
     )

Commit message: feat: updated BOM
Parts:
- C26, C28: value (none) -> 100n; footprint (none) -> Capacitor_SMD:C_0805_2012Metric_Pad1.18x1.45mm_HandSolder
- C27, C29: value (none) -> 10u; footprint (none) -> Capacitor_SMD:C_0805_2012Metric_Pad1.18x1.45mm_HandSolder
- J8: value (none) -> SJ
- R41: value (none) -> 10k
- SJ1: value (none) -> JUMPER-PAD-2-NC_BY_TRACE
- U6: value (none) -> HX711
Changed lines of the file:
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@@
       (effects (font (size 1.4986 1.4986)) (justify right))
     )
-    (property "Value" "" (id 1) (at 82.55 106.68 0)
+    (property "Value" "JUMPER-PAD-2-NC_BY_TRACE" (id 1) (at 82.55 106.68 0)
       (effects (font (size 1.4986 1.4986)) (justify right))
     )
@@
       (effects (font (size 1.27 1.27)) (justify left))
     )
-    (property "Value" "" (id 1) (at 97.155 126.365 0)
+    (property "Value" "100n" (id 1) (at 97.155 126.365 0)
       (effects (font (size 1.27 1.27)) (justify left))
     )
-    (property "Footprint" "" (id 2) (at 97.4852 127.635 0)
+    (property "Footprint" "Capacitor_SMD:C_0805_2012Metric_Pad1.18x1.45mm_HandSolder" (id 2) (at 97.4852 127.635 0)
       (effects (font (size 1.27 1.27)) hide)
     )
@@
       (effects (font (size 1.27 1.27)) (justify left))
     )
-    (property "Value" "" (id 1) (at 105.41 126.365 0)
+    (property "Value" "10u" (id 1) (at 105.41 126.365 0)
       (effects (font (size 1.27 1.27)) (justify left))
     )
-    (property "Footprint" "" (id 2) (at 105.7402 127.635 0)
+    (property "Footprint" "Capacitor_SMD:C_0805_2012Metric_Pad1.18x1.45mm_HandSolder" (id 2) (at 105.7402 127.635 0)
       (effects (font (size 1.27 1.27)) hide)
     )
@@
       (effects (font (size 1.27 1.27)) (justify left))
     )
-    (property "Value" "" (id 1) (at 123.19 90.17 0)
+    (property "Value" "100n" (id 1) (at 123.19 90.17 0)
       (effects (font (size 1.27 1.27)) (justify left))
     )
-    (property "Footprint" "" (id 2) (at 123.5202 91.44 0)
+    (property "Footprint" "Capacitor_SMD:C_0805_2012Metric_Pad1.18x1.45mm_HandSolder" (id 2) (at 123.5202 91.44 0)
       (effects (font (size 1.27 1.27)) hide)
     )
@@
       (effects (font (size 1.27 1.27)) (justify left))
     )
-    (property "Value" "" (id 1) (at 131.445 90.17 0)
+    (property "Value" "10u" (id 1) (at 131.445 90.17 0)
       (effects (font (size 1.27 1.27)) (justify left))
     )
-    (property "Footprint" "" (id 2) (at 131.7752 91.44 0)
+    (property "Footprint" "Capacitor_SMD:C_0805_2012Metric_Pad1.18x1.45mm_HandSolder" (id 2) (at 131.7752 91.44 0)
       (effects (font (size 1.27 1.27)) hide)
     )
@@
       (effects (font (size 1.4986 1.4986)))
     )
-    (property "Value" "" (id 1) (at 198.755 78.74 0)
+    (property "Value" "SJ" (id 1) (at 198.755 78.74 0)
       (effects (font (size 1.4986 1.4986)))
     )
@@
       (effects (font (size 1.27 1.27)) (justify left))
     )
-    (property "Value" "" (id 1) (at 192.405 73.025 90)
+    (property "Value" "10k" (id 1) (at 192.405 73.025 90)
       (effects (font (size 1.27 1.27)) (justify left))
     )
@@
       (effects (font (size 1.4986 1.4986)))
     )
-    (property "Value" "" (id 1) (at 169.545 66.5226 0)
+    (property "Value" "HX711" (id 1) (at 169.545 66.5226 0)
       (effects (font (size 1.4986 1.4986)))
     )
