File: pcb/main/Memory.kicad_sch (KiCad schematic)
At the start: 5 parts

Commit message: feat: updated BOM
Parts:
- C31: value (none) -> 10u; footprint (none) -> Capacitor_SMD:C_0805_2012Metric_Pad1.18x1.45mm_HandSolder
- R42, R43, R44: value (none) -> 1k
- U7: value (none) -> SST26VF064B
Changed lines of the file:
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@@
     (in_bom yes) (on_board yes)
     (property "Reference" "R44" (id 0) (at 112.395 57.785 90))
-    (property "Value" "" (id 1) (at 120.65 60.325 90))
+    (property "Value" "1k" (id 1) (at 120.65 60.325 90))
     (property "Footprint" "" (id 2) (at 116.84 57.277 90)
       (effects (font (size 1.27 1.27)) hide)
@@
     (in_bom yes) (on_board yes)
     (property "Reference" "R43" (id 0) (at 112.395 55.245 90))
-    (property "Value" "" (id 1) (at 120.65 57.785 90))
+    (property "Value" "1k" (id 1) (at 120.65 57.785 90))
     (property "Footprint" "" (id 2) (at 116.84 54.737 90)
       (effects (font (size 1.27 1.27)) hide)
@@
       (effects (font (size 1.27 1.27)) (justify right))
     )
-    (property "Value" "" (id 1) (at 100.457 50.038 0)
+    (property "Value" "1k" (id 1) (at 100.457 50.038 0)
       (effects (font (size 1.27 1.27)) (justify right))
     )
@@
       (effects (font (size 1.27 1.27)) (justify left))
     )
-    (property "Value" "" (id 1) (at 115.316 39.878 0)
+    (property "Value" "10u" (id 1) (at 115.316 39.878 0)
       (effects (font (size 1.27 1.27)) (justify left))
     )
-    (property "Footprint" "" (id 2) (at 113.3602 42.545 0)
+    (property "Footprint" "Capacitor_SMD:C_0805_2012Metric_Pad1.18x1.45mm_HandSolder" (id 2) (at 113.3602 42.545 0)
       (effects (font (size 1.27 1.27)) hide)
     )
@@
       (effects (font (size 1.27 1.27)) (justify left))
     )
-    (property "Value" "" (id 1) (at 144.6276 60.198 0)
+    (property "Value" "SST26VF064B" (id 1) (at 144.6276 60.198 0)
       (effects (font (size 1.27 1.27)) (justify left))
     )
