File: pcb/main/pHMeter.kicad_sch (KiCad schematic)
At the start: 86 parts

Commit message: fix: symbol libraries in Kicad 6.0
Parts:
- C11, C20, C23, C6: value (none) -> 10u; footprint (none) -> Capacitor_SMD:C_0805_2012Metric_Pad1.15x1.40mm_HandSolder; symbol pHMeter-rescue:C-Device -> Device:C
- C13, C14: value (none) -> 18p; footprint (none) -> Capacitor_SMD:C_0805_2012Metric_Pad1.15x1.40mm_HandSolder; symbol pHMeter-rescue:C-Device -> Device:C
- C15, C16, C17, C33, C7: value (none) -> 100n; footprint (none) -> Capacitor_SMD:C_0805_2012Metric_Pad1.15x1.40mm_HandSolder; symbol pHMeter-rescue:C-Device -> Device:C
- C18: value (none) -> 1u; footprint (none) -> Capacitor_SMD:C_0805_2012Metric_Pad1.15x1.40mm_HandSolder; symbol pHMeter-rescue:C-Device -> Device:C
- C21: symbol pHMeter-rescue:C-Device -> Device:C
- D11, D19, D9: value (none) -> YELLOW; footprint (none) -> LED_SMD:LED_0805_2012Metric_Pad1.15x1.40mm_HandSolder; symbol pHMeter-rescue:LED-Device -> Device:LED
- D12, D17, D18: value (none) -> BLUE; footprint (none) -> LED_SMD:LED_0805_2012Metric_Pad1.15x1.40mm_HandSolder; symbol pHMeter-rescue:LED-Device -> Device:LED
- D13: symbol pHMeter-rescue:LED-Device -> Device:LED
- D14: symbol pHMeter-rescue:D_Schottky-Device -> Device:D_Schottky
- D3, D4, D5: value (none) -> MBR0520LT1G; footprint (none) -> Diode_SMD:D_SOD-123; symbol pHMeter-rescue:D_Schottky-Device -> Device:D_Schottky
- D7, D8: value (none) -> GREEN; footprint (none) -> LED_SMD:LED_0805_2012Metric_Pad1.15x1.40mm_HandSolder; symbol pHMeter-rescue:LED-Device -> Device:LED
- DS1: symbol pHMeter-rescue:WC1602A-Display_Character -> Display_Character:WC1602A
- H1: symbol pHMeter-rescue:MountingHole-Mechanical -> Mechanical:MountingHole
- H2, H3, H4: value (none) -> MountingHole; footprint (none) -> MountingHole:MountingHole_3.2mm_M3; symbol pHMeter-rescue:MountingHole-Mechanical -> Mechanical:MountingHole
- J1: symbol pHMeter-rescue:Conn_02x03_Odd_Even-Connector_Generic -> Connector_Generic:Conn_02x03_Odd_Even
- J4: symbol pHMeter-rescue:AudioJack3_SwitchTR-Connector -> Connector:AudioJack3_SwitchTR
- J5: symbol pHMeter-rescue:RJ12-Connector -> Connector:RJ12
- J6: value (none) -> AudioJack3_SwitchTR; footprint (none) -> Connector_Audio:Jack_3.5mm_Ledino_KB3SPRS_Horizontal; symbol pHMeter-rescue:AudioJack3_SwitchTR-Connector -> Connector:AudioJack3_SwitchTR
- J7: value (none) -> SJ; footprint (none) -> Jumper:SolderJumper-2_P1.3mm_Open_RoundedPad1.0x1.5mm
- JP1, JP2: value (none) -> JP1E; footprint (none) -> Connector_PinHeader_2.54mm:PinHeader_1x02_P2.54mm_Vertical
- JP3: value (none) -> acidic; footprint (none) -> Connector_Molex:Molex_KK-254_AE-6410-02A_1x02_P2.54mm_Vertical
- JP4: value (none) -> alkaline; footprint (none) -> Connector_Molex:Molex_KK-254_AE-6410-02A_1x02_P2.54mm_Vertical
- JP5: value (none) -> Bat; footprint (none) -> Connector_Molex:Molex_KK-254_AE-6410-02A_1x02_P2.54mm_Vertical
- JP6: value (none) -> IO3; footprint (none) -> Connector_Molex:Molex_KK-254_AE-6410-02A_1x02_P2.54mm_Vertical
- JP7: value (none) -> IO4; footprint (none) -> Connector_Molex:Molex_KK-254_AE-6410-02A_1x02_P2.54mm_Vertical
- Q1, Q2, Q4, Q5: value (none) -> ZXMS6004; footprint (none) -> Package_TO_SOT_SMD:SOT-23
- Q3: value (none) -> DMP1045; footprint (none) -> Package_TO_SOT_SMD:SOT-23
- R14, R15: value (none) -> 22; footprint (none) -> Resistor_SMD:R_0805_2012Metric_Pad1.15x1.40mm_HandSolder; symbol pHMeter-rescue:R-Device -> Device:R
- R16, R25, R26, R27, R28, R30, R34, R36, R37, R47, R48: value (none) -> 10k; footprint (none) -> Resistor_SMD:R_0805_2012Metric_Pad1.15x1.40mm_HandSolder; symbol pHMeter-rescue:R-Device -> Device:R
- R19, R20, R23, R24, R49, R55: value (none) -> 1k; footprint (none) -> Resistor_SMD:R_0805_2012Metric_Pad1.15x1.40mm_HandSolder; symbol pHMeter-rescue:R-Device -> Device:R
- R21, R51: value (none) -> 4.7k; footprint (none) -> Resistor_SMD:R_0805_2012Metric_Pad1.15x1.40mm_HandSolder; symbol pHMeter-rescue:R-Device -> Device:R
- R22, R32, R33, R53: value (none) -> 100; footprint (none) -> Resistor_SMD:R_0805_2012Metric_Pad1.15x1.40mm_HandSolder; symbol pHMeter-rescue:R-Device -> Device:R
- R29: symbol pHMeter-rescue:R-Device -> Device:R
- R31: value (none) -> 0; footprint (none) -> Resistor_SMD:R_0805_2012Metric_Pad1.15x1.40mm_HandSolder; symbol pHMeter-rescue:R-Device -> Device:R
- R35, R38, R45: value (none) -> 1M; footprint (none) -> Resistor_SMD:R_0805_2012Metric_Pad1.15x1.40mm_HandSolder; symbol pHMeter-rescue:R-Device -> Device:R
- R46: value (none) -> 100k; footprint (none) -> Resistor_SMD:R_0805_2012Metric_Pad1.15x1.40mm_HandSolder; symbol pHMeter-rescue:R-Device -> Device:R
- RV1: symbol pHMeter-rescue:R_POT-Device -> Device:R_Potentiometer
- SW1: symbol pHMeter-rescue:Rotary_Encoder_Switch-Device -> Device:RotaryEncoder_Switch
- U3: value (none) -> ATMEGA32U4-AU; footprint (none) -> Package_QFP:TQFP-44_10x10mm_P0.8mm
- U4: symbol pHMeter-rescue:MCP1703A-1202_SOT23-Regulator_Linear -> Regulator_Linear:MCP1703A-1202_SOT23
- U9: symbol pHMeter-rescue:MCP73811T-420I-OT-Battery_Management -> Battery_Management:MCP73811T-420I-OT
- X1: value (none) -> MINI-USB-SCHIELD-32005-201; footprint (none) -> Connector_USB:USB_Mini-B_Lumberg_2486_01_Horizontal
- Y1: symbol pHMeter-rescue:Crystal-Device -> Device:Crystal
Connections:
- net +12V: now also C20.1, J5.1, R16.1, U4.3 (VI)
- net A2: now also R47.1
- net A3: now also R48.1
- net A4: now also C33.1, R38.2, R45.1
- net A6: now also DS1.4 (RS)
- net AREF: now also C16.1
- net D10: now also DS1.13 (D6)
- net D11: now also R26.1
- net D12: now also R27.1
- net D13: now also DS1.2 (VDD), R20.1, R31.1, R32.1
- net D5: now also DS1.14 (D7)
- net D6: now also DS1.6 (E)
- net D7: now also SW1.S1
- net D8: now also DS1.11 (D4)
- net D9: now also DS1.12 (D5)
- net GND: now also C11.2, C13.2, C14.2, C15.1, C16.2, C17.2, C18.2, C20.2, C21.1, C23.2, C33.2, C6.2, C7.2, D12.1 (K), D13.1 (K), D17.1 (K), D18.1 (K), D7.1 (K), D8.1 (K), DS1.1 (VSS), DS1.16 (LED(-)), DS1.5 (R/W), J1.6 (Pin_6), J4.R, J5.4, J5.6, J6.R, R33.2, R36.1, R37.1, R45.2, R46.2, SW1.C, SW1.S2, U4.1 (GND), U9.2 (VSS)
- net HWB: now also R36.2
- net MISO: now also J1.1 (Pin_1)
- net MOSI: now also J1.4 (Pin_4)
- net ONE-WIRE-1: now also R49.1
- net ONE-WIRE-2: now also R19.1
- net RESET: now also J1.5 (Pin_5), R34.2
- net RX: now also SW1.B
- net SCK: now also J1.3 (Pin_3)
- net SCL: now also J5.2, R28.2
- net SDA: now also J5.3, R25.2
- net TX: now also D11.1 (K), SW1.A
- net USB_N: now also R14.1
- net USB_P: now also R15.1
- net VBAT: now also D14.1 (K)
- net VDD: now also C21.2, D14.2 (A), D3.1 (K), D4.1 (K), D5.1 (K), R29.2, R46.1, U9.4 (VDD)
- net VUSB: now also C11.1, D4.2 (A)
- net at X1.2: now also R14.2
- net at X1.3: now also R15.2
- net at JP5.1, Q3.3 (D): now also C23.1, R38.1, U9.3 (VBAT)
- net at U3.16 (XTAL2): now also C14.1, Y1.2
- net at U3.17 (XTAL1): now also C13.1, Y1.1
- net at U3.6 (UCAP): now also C18.1
- net 3.3V renamed +3V3
- net +3V3: now also C17.1, R22.2, R23.2, R24.1, R25.1, R28.1, R34.1, R53.2, R55.2
- new net: D3.2 (A), J1.2 (Pin_2)
- new net: C6.1, C7.1, D5.2 (A), U4.2 (VO)
- new net: D11.2 (A), R24.2
- new net: D8.2 (A), R20.2
- new net: DS1.15 (LED(+)), R31.2
- new net: DS1.3 (VO), RV1.2
- new net: D12.2 (A), R27.2
- new net: D13.2 (A), R26.2
- new net: D7.2 (A), R16.2
- new net: R33.1, RV1.1
- new net: R32.2, RV1.3
- new net: R30.1, U9.1 (CEN)
- new net: R37.2, U9.5 (PROG)
- new net: R29.1, R30.2
- new net: D17.2 (A), R47.2
- new net: D18.2 (A), R48.2
- new net: D19.2 (A), R55.1
- new net: D19.1 (K), J4.S, R51.2, R53.1
- new net: J4.T, R49.2, R51.1
- new net: D9.2 (A), R23.1
- new net: D9.1 (K), J6.S, R21.2, R22.1
- new net: J6.T, R19.2, R21.1

Commit message: fix: 3D model libraries in Kicad 6.0
Parts:
- C21: value (none) -> 10u; footprint (none) -> Capacitor_SMD:C_0805_2012Metric_Pad1.15x1.40mm_HandSolder
- D13: value (none) -> BLUE; footprint (none) -> LED_SMD:LED_0805_2012Metric_Pad1.15x1.40mm_HandSolder
- D14: value (none) -> MBR0520LT1G; footprint (none) -> Diode_SMD:D_SOD-123
- DS1: value (none) -> WC1602A; footprint (none) -> Display:WC1602A
- H1: value (none) -> MountingHole; footprint (none) -> MountingHole:MountingHole_3.2mm_M3
- J1: value (none) -> Conn_02x03_Odd_Even; footprint (none) -> Connector:Tag-Connect_TC2030-IDC-NL_2x03_P1.27mm_Vertical
- J4: value (none) -> AudioJack3_SwitchTR; footprint (none) -> Connector_Audio:Jack_3.5mm_Ledino_KB3SPRS_Horizontal
- J5: value (none) -> RJ12; footprint (none) -> pHMeter:E5566-Q0LK22-L
- R29: value (none) -> 10k; footprint (none) -> Resistor_SMD:R_0805_2012Metric_Pad1.20x1.40mm_HandSolder
- RV1: value (none) -> 10k; footprint (none) -> Potentiometer_THT:Potentiometer_Bourns_3339P_Vertical_HandSoldering
- SW1: value (none) -> Rotary_Encoder_Switch; footprint (none) -> Rotary_Encoder:RotaryEncoder_Alps_EC11E-Switch_Vertical_H20mm
- U4: value (none) -> MCP1703A; footprint (none) -> Package_TO_SOT_SMD:SOT-23
- U9: value (none) -> MCP73811T; footprint (none) -> Package_TO_SOT_SMD:SOT-23-5
- Y1: value (none) -> Crystal; footprint (none) -> Crystal:Crystal_SMD_0603-2Pin_6.0x3.5mm_HandSoldering

Commit message: fix: standard footprint for R and C, BOM updated
Parts:
- C11, C20, C21, C23: value 10u -> (none); footprint Capacitor_SMD:C_0805_2012Metric_Pad1.15x1.40mm_HandSolder -> (none); MFN Samsung Electro-Mechanics -> Wurth Elektronik; MFP CL21A106KOQNNNG -> 885012207072; S1PL https://www.mouser.com/ProductDetail/Samsung-Electro-Mechan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 -> https://www.mouser.com/ProductDetail/Wurth-Elektronik/88501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; S1PN 187-CL21A106KOQNNNG -> 710-885012207072
- C13, C14: value 18p -> (none); footprint Capacitor_SMD:C_0805_2012Metric_Pad1.15x1.40mm_HandSolder -> (none)
- C15, C16, C17, C33: value 100n -> (none); footprint Capacitor_SMD:C_0805_2012Metric_Pad1.15x1.40mm_HandSolder -> (none)
- C18: value 1u -> (none); footprint Capacitor_SMD:C_0805_2012Metric_Pad1.15x1.40mm_HandSolder -> (none)
- C6: value 10u -> (none); footprint Capacitor_SMD:C_0805_2012Metric_Pad1.15x1.40mm_HandSolder -> (none)
- C7: value 100n -> (none); footprint Capacitor_SMD:C_0805_2012Metric_Pad1.15x1.40mm_HandSolder -> (none); MFN Samsung Electro-Mechanics -> Wurth Elektronik; MFP CL21A106KOQNNNG -> 885012207072; S1PL https://www.mouser.com/ProductDetail/Samsung-Electro-Mechan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 -> https://www.mouser.com/ProductDetail/Wurth-Elektronik/88501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; S1PN 187-CL21A106KOQNNNG -> 710-885012207072
- D11, D19, D9: value YELLOW -> (none); footprint LED_SMD:LED_0805_2012Metric_Pad1.15x1.40mm_HandSolder -> (none)
- D12, D13, D17, D18: value BLUE -> (none); footprint LED_SMD:LED_0805_2012Metric_Pad1.15x1.40mm_HandSolder -> (none)
- D14, D3, D4, D5: value MBR0520LT1G -> (none); footprint Diode_SMD:D_SOD-123 -> (none)
- D7, D8: value GREEN -> (none); footprint LED_SMD:LED_0805_2012Metric_Pad1.15x1.40mm_HandSolder -> (none)
- DS1: value WC1602A -> (none); footprint Display:WC1602A -> (none)
- H1, H2, H3, H4: value MountingHole -> (none); footprint MountingHole:MountingHole_3.2mm_M3 -> (none)
- J1: value Conn_02x03_Odd_Even -> (none); footprint Connector:Tag-Connect_TC2030-IDC-NL_2x03_P1.27mm_Vertical -> (none)
- J4, J6: value AudioJack3_SwitchTR -> (none); footprint Connector_Audio:Jack_3.5mm_Ledino_KB3SPRS_Horizontal -> (none)
- J5: value RJ12 -> (none); footprint pHMeter:E5566-Q0LK22-L -> (none)
- J7: value SJ -> (none); footprint Jumper:SolderJumper-2_P1.3mm_Open_RoundedPad1.0x1.5mm -> (none)
- JP1, JP2: value JP1E -> (none); footprint Connector_PinHeader_2.54mm:PinHeader_1x02_P2.54mm_Vertical -> (none)
- JP3: value acidic -> (none); footprint Connector_Molex:Molex_KK-254_AE-6410-02A_1x02_P2.54mm_Vertical -> (none)
- JP4: value alkaline -> (none); footprint Connector_Molex:Molex_KK-254_AE-6410-02A_1x02_P2.54mm_Vertical -> (none)
- JP5: value Bat -> (none); footprint Connector_Molex:Molex_KK-254_AE-6410-02A_1x02_P2.54mm_Vertical -> (none)
- JP6: value IO3 -> (none); footprint Connector_Molex:Molex_KK-254_AE-6410-02A_1x02_P2.54mm_Vertical -> (none)
- JP7: value IO4 -> (none); footprint Connector_Molex:Molex_KK-254_AE-6410-02A_1x02_P2.54mm_Vertical -> (none)
- Q1, Q2, Q4, Q5: value ZXMS6004 -> (none); footprint Package_TO_SOT_SMD:SOT-23 -> (none)
- Q3: value DMP1045 -> (none); footprint Package_TO_SOT_SMD:SOT-23 -> (none)
- R14, R15: value 22 -> (none); footprint Resistor_SMD:R_0805_2012Metric_Pad1.15x1.40mm_HandSolder -> (none)
- R16, R25, R26, R27, R28, R30, R34, R36, R37, R47, R48: value 10k -> (none); footprint Resistor_SMD:R_0805_2012Metric_Pad1.15x1.40mm_HandSolder -> (none)
- R19, R20, R23, R24, R49, R55: value 1k -> (none); footprint Resistor_SMD:R_0805_2012Metric_Pad1.15x1.40mm_HandSolder -> (none)
- R21, R51: value 4.7k -> (none); footprint Resistor_SMD:R_0805_2012Metric_Pad1.15x1.40mm_HandSolder -> (none)
- R22, R32, R33, R53: value 100 -> (none); footprint Resistor_SMD:R_0805_2012Metric_Pad1.15x1.40mm_HandSolder -> (none)
- R29: value 10k -> (none); footprint Resistor_SMD:R_0805_2012Metric_Pad1.20x1.40mm_HandSolder -> (none)
- R31: value 0 -> (none); footprint Resistor_SMD:R_0805_2012Metric_Pad1.15x1.40mm_HandSolder -> (none)
- R35, R38, R45: value 1M -> (none); footprint Resistor_SMD:R_0805_2012Metric_Pad1.15x1.40mm_HandSolder -> (none)
- R46: value 100k -> (none); footprint Resistor_SMD:R_0805_2012Metric_Pad1.15x1.40mm_HandSolder -> (none)
- RV1: value 10k -> (none); footprint Potentiometer_THT:Potentiometer_Bourns_3339P_Vertical_HandSoldering -> (none)
- SW1: value Rotary_Encoder_Switch -> (none); footprint Rotary_Encoder:RotaryEncoder_Alps_EC11E-Switch_Vertical_H20mm -> (none)
- U3: value ATMEGA32U4-AU -> (none); footprint Package_QFP:TQFP-44_10x10mm_P0.8mm -> (none)
- U4: value MCP1703A -> (none); footprint Package_TO_SOT_SMD:SOT-23 -> (none)
- U9: value MCP73811T -> (none); footprint Package_TO_SOT_SMD:SOT-23-5 -> (none)
- X1: value MINI-USB-SCHIELD-32005-201 -> (none); footprint Connector_USB:USB_Mini-B_Lumberg_2486_01_Horizontal -> (none)
- Y1: value Crystal -> (none); footprint Crystal:Crystal_SMD_0603-2Pin_6.0x3.5mm_HandSoldering -> (none)

Commit message: feat: updated BOM
BOM ready to order in v0.2
Parts:
- C11, C20, C21, C23, C6: value (none) -> 10u; footprint (none) -> Capacitor_SMD:C_0805_2012Metric_Pad1.18x1.45mm_HandSolder; MFN Wurth Elektronik -> Samsung Electro-Mechanics; MFP 885012207072 -> CL21A106KOQNNNG; S1PL https://www.mouser.com/ProductDetail/Wurth-Elektronik/88501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 -> https://www.mouser.com/ProductDetail/Samsung-Electro-Mechan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; S1PN 710-885012207072 -> 187-CL21A106KOQNNNG
- C13, C14: value (none) -> 18p; footprint (none) -> Capacitor_SMD:C_0805_2012Metric_Pad1.15x1.40mm_HandSolder
- C15, C16, C17, C33, C7: value (none) -> 100n; footprint (none) -> Capacitor_SMD:C_0805_2012Metric_Pad1.18x1.45mm_HandSolder
- C18: value (none) -> 1u; footprint (none) -> Capacitor_SMD:C_0805_2012Metric_Pad1.15x1.40mm_HandSolder
- D11, D19, D9: value (none) -> YELLOW; footprint (none) -> LED_SMD:LED_0805_2012Metric_Pad1.15x1.40mm_HandSolder
- D12, D13, D17, D18: value (none) -> BLUE; footprint (none) -> LED_SMD:LED_0805_2012Metric_Pad1.15x1.40mm_HandSolder
- D14, D3, D4, D5: value (none) -> MBR0520LT1G; footprint (none) -> Diode_SMD:D_SOD-123
- D7, D8: value (none) -> GREEN; footprint (none) -> LED_SMD:LED_0805_2012Metric_Pad1.15x1.40mm_HandSolder
- DS1: value (none) -> WC1602A; footprint (none) -> Display:WC1602A
- H1, H2, H3, H4: value (none) -> MountingHole; footprint (none) -> MountingHole:MountingHole_3.2mm_M3
- J1: value (none) -> Conn_02x03_Odd_Even; footprint (none) -> Connector:Tag-Connect_TC2030-IDC-NL_2x03_P1.27mm_Vertical
- J4, J6: value (none) -> AudioJack3_SwitchTR; footprint (none) -> Connector_Audio:Jack_3.5mm_Ledino_KB3SPRS_Horizontal
- J5: value (none) -> RJ12; footprint (none) -> pHMeter:E5566-Q0LK22-L
- J7: value (none) -> SJ; footprint (none) -> Jumper:SolderJumper-2_P1.3mm_Open_RoundedPad1.0x1.5mm
- JP1, JP2: value (none) -> JP1E; footprint (none) -> Connector_PinHeader_2.54mm:PinHeader_1x02_P2.54mm_Vertical
- JP3: value (none) -> acidic; footprint (none) -> Connector_Molex:Molex_KK-254_AE-6410-02A_1x02_P2.54mm_Vertical
- JP4: value (none) -> alkaline; footprint (none) -> Connector_Molex:Molex_KK-254_AE-6410-02A_1x02_P2.54mm_Vertical
- JP5: value (none) -> Bat; footprint (none) -> Connector_Molex:Molex_KK-254_AE-6410-02A_1x02_P2.54mm_Vertical
- JP6: value (none) -> IO3; footprint (none) -> Connector_Molex:Molex_KK-254_AE-6410-02A_1x02_P2.54mm_Vertical
- JP7: value (none) -> IO4; footprint (none) -> Connector_Molex:Molex_KK-254_AE-6410-02A_1x02_P2.54mm_Vertical
- Q1, Q2, Q4, Q5: value (none) -> ZXMS6004; footprint (none) -> Package_TO_SOT_SMD:SOT-23
- Q3: value (none) -> DMP1045; footprint (none) -> Package_TO_SOT_SMD:SOT-23
- R14, R15: value (none) -> 22; footprint (none) -> Resistor_SMD:R_0805_2012Metric_Pad1.15x1.40mm_HandSolder
- R16, R25, R26, R27, R28, R29, R30, R34, R36, R37, R47, R48: value (none) -> 10k; footprint (none) -> Resistor_SMD:R_0805_2012Metric_Pad1.20x1.40mm_HandSolder
- R19, R20, R23, R24, R49, R55: value (none) -> 1k; footprint (none) -> Resistor_SMD:R_0805_2012Metric_Pad1.15x1.40mm_HandSolder
- R21, R51: value (none) -> 4.7k; footprint (none) -> Resistor_SMD:R_0805_2012Metric_Pad1.15x1.40mm_HandSolder
- R22, R32, R33, R53: value (none) -> 100; footprint (none) -> Resistor_SMD:R_0805_2012Metric_Pad1.15x1.40mm_HandSolder
- R31: value (none) -> 0; footprint (none) -> Resistor_SMD:R_0805_2012Metric_Pad1.15x1.40mm_HandSolder
- R35, R38, R45: value (none) -> 1M; footprint (none) -> Resistor_SMD:R_0805_2012Metric_Pad1.15x1.40mm_HandSolder
- R46: value (none) -> 100k; footprint (none) -> Resistor_SMD:R_0805_2012Metric_Pad1.20x1.40mm_HandSolder
- RV1: value (none) -> 10k; footprint (none) -> Potentiometer_THT:Potentiometer_Bourns_3339P_Vertical_HandSoldering
- SW1: value (none) -> Rotary_Encoder_Switch; footprint (none) -> Rotary_Encoder:RotaryEncoder_Alps_EC11E-Switch_Vertical_H20mm
- U3: value (none) -> ATMEGA32U4-AU; footprint (none) -> Package_QFP:TQFP-44_10x10mm_P0.8mm
- U4: value (none) -> MCP1703A; footprint (none) -> Package_TO_SOT_SMD:SOT-23
- U9: value (none) -> MCP73811T; footprint (none) -> Package_TO_SOT_SMD:SOT-23-5
- X1: value (none) -> MINI-USB-SCHIELD-32005-201; footprint (none) -> Connector_USB:USB_Mini-B_Lumberg_2486_01_Horizontal
- Y1: value (none) -> Crystal; footprint (none) -> Crystal:Crystal_SMD_0603-2Pin_6.0x3.5mm_HandSoldering

Commit message: feat: new PCB version to 1.1.2
Schematic:
- Updated sheets to 1.1.2 version.
- Change inputs for last OPA in EC sheet.
- INA- and INA+ set to GND in 24bits sheet for reduce noise.
- Change /CE connection (TX -> HWB) in Memory and COMM LED.
- Adding a correct guard in pH sheet.
- Adding correct 12 V support for 3.3 V (avoid battery charge circuit).

Design:
- Increase width track for 2 A in 3.3 V power supply.
- Order labels.
- Put new schottky diode for 12 V -> 3.3 V circuit direct connection.
- Adding pH and EC tag.
- Adding guard and restrict area for pH adquisiton.
Parts:
- added D10: MBR0520LT1G, Diode_SMD:D_SOD-123, symbol Device:D_Schottky
Connections:
- net +12V: now also D10.2 (A)
- net HWB: now also D11.1 (K)
- net RESET: now also C15.2
- net TX: no longer D11.1 (K)
- net VBAT: now also D10.1 (K)
- net at R35.1: now also C13.1, U3.17 (XTAL1), Y1.1
- net at R35.2: now also C14.1, U3.16 (XTAL2), Y1.2
Other:
- moved on the sheet: C15, J7
Changed lines of the file:
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@@
   (title_block
     (title "PHMeter")
-    (date "2021-11-29")
-    (rev "1.0")
+    (date "2022-07-25")
+    (rev "1.1.2")
     (company "Hackuarium")
     (comment 1 "New version for pH and conductivity Meter")
+    (comment 2 "New connections in EC for last OPA")
   )

Commit message: feat: updated BOM information
Some components are still without MNF and Seller information
Parts:
- C11, C20, C21, C23, C6: value 10u -> (none); footprint Capacitor_SMD:C_0805_2012Metric_Pad1.18x1.45mm_HandSolder -> (none)
- C13, C14: value 18p -> (none); footprint Capacitor_SMD:C_0805_2012Metric_Pad1.15x1.40mm_HandSolder -> (none)
- C15, C16, C17, C33, C7: value 100n -> (none); footprint Capacitor_SMD:C_0805_2012Metric_Pad1.18x1.45mm_HandSolder -> (none)
- C18: value 1u -> (none); footprint Capacitor_SMD:C_0805_2012Metric_Pad1.15x1.40mm_HandSolder -> (none)
- D10, D14, D3, D4, D5: value MBR0520LT1G -> (none); footprint Diode_SMD:D_SOD-123 -> (none)
- D11, D19, D9: value YELLOW -> (none); footprint LED_SMD:LED_0805_2012Metric_Pad1.15x1.40mm_HandSolder -> (none)
- D12, D13, D17, D18: value BLUE -> (none); footprint LED_SMD:LED_0805_2012Metric_Pad1.15x1.40mm_HandSolder -> (none)
- D7, D8: value GREEN -> (none); footprint LED_SMD:LED_0805_2012Metric_Pad1.15x1.40mm_HandSolder -> (none)
- DS1: value WC1602A -> (none); footprint Display:WC1602A -> (none)
- H1, H2, H3, H4: value MountingHole -> (none); footprint MountingHole:MountingHole_3.2mm_M3 -> (none)
- J1: value Conn_02x03_Odd_Even -> (none); footprint Connector:Tag-Connect_TC2030-IDC-NL_2x03_P1.27mm_Vertical -> (none)
- J4, J6: value AudioJack3_SwitchTR -> (none); footprint Connector_Audio:Jack_3.5mm_Ledino_KB3SPRS_Horizontal -> (none)
- J5: value RJ12 -> (none); footprint pHMeter:E5566-Q0LK22-L -> (none)
- J7: value SJ -> (none); footprint Jumper:SolderJumper-2_P1.3mm_Open_RoundedPad1.0x1.5mm -> (none)
- JP1, JP2: value JP1E -> (none); footprint Connector_PinHeader_2.54mm:PinHeader_1x02_P2.54mm_Vertical -> (none)
- JP3: value acidic -> (none); footprint Connector_Molex:Molex_KK-254_AE-6410-02A_1x02_P2.54mm_Vertical -> (none)
- JP4: value alkaline -> (none); footprint Connector_Molex:Molex_KK-254_AE-6410-02A_1x02_P2.54mm_Vertical -> (none)
- JP5: value Bat -> (none); footprint Connector_Molex:Molex_KK-254_AE-6410-02A_1x02_P2.54mm_Vertical -> (none)
- JP6: value IO3 -> (none); footprint Connector_Molex:Molex_KK-254_AE-6410-02A_1x02_P2.54mm_Vertical -> (none)
- JP7: value IO4 -> (none); footprint Connector_Molex:Molex_KK-254_AE-6410-02A_1x02_P2.54mm_Vertical -> (none)
- Q1, Q2, Q4, Q5: value ZXMS6004 -> (none); footprint Package_TO_SOT_SMD:SOT-23 -> (none); MFN (none) -> Diodes Incorporated; MFP (none) -> ZXMS6004FFTA; S1PL (none) -> https://www.mouser.com/ProductDetail/Diodes-Incorporated/ZX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; S1PN (none) -> 522-ZXMS6004FFTA
- Q3: value DMP1045 -> (none); footprint Package_TO_SOT_SMD:SOT-23 -> (none)
- R14, R15: value 22 -> (none); footprint Resistor_SMD:R_0805_2012Metric_Pad1.15x1.40mm_HandSolder -> (none)
- R16, R25, R26, R27, R28, R29, R30, R34, R36, R37, R47, R48: value 10k -> (none); footprint Resistor_SMD:R_0805_2012Metric_Pad1.20x1.40mm_HandSolder -> (none)
- R19, R20, R23, R24, R49, R55: value 1k -> (none); footprint Resistor_SMD:R_0805_2012Metric_Pad1.15x1.40mm_HandSolder -> (none); MFN (none) -> KOA Speer; MFP (none) -> RK73H2ATTD1001F; S1PL (none) -> https://www.mouser.com/ProductDetail/KOA-Speer/RK73H2ATTD10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; S1PN (none) -> 660-RK73H2ATTD1001F
- R21, R51: value 4.7k -> (none); footprint Resistor_SMD:R_0805_2012Metric_Pad1.15x1.40mm_HandSolder -> (none)
- R22, R32, R33, R53: value 100 -> (none); footprint Resistor_SMD:R_0805_2012Metric_Pad1.15x1.40mm_HandSolder -> (none); MFN (none) -> KOA Speer; MFP (none) -> RK73H2ATTD1000F; S1PL (none) -> https://www.mouser.com/ProductDetail/KOA-Speer/RK73H2ATTD10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; S1PN (none) -> 660-RK73H2ATTD1000F
- R31: value 0 -> (none); footprint Resistor_SMD:R_0805_2012Metric_Pad1.15x1.40mm_HandSolder -> (none)
- R35, R38, R45: value 1M -> (none); footprint Resistor_SMD:R_0805_2012Metric_Pad1.15x1.40mm_HandSolder -> (none)
- R46: value 100k -> (none); footprint Resistor_SMD:R_0805_2012Metric_Pad1.20x1.40mm_HandSolder -> (none); MFN (none) -> Vishay / Dale; MFP (none) -> CRCW0805100KJNEC; S1PL (none) -> https://www.mouser.com/ProductDetail/Vishay-Dale/CRCW080510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; S1PN (none) -> 71-CRCW0805100KJNEC
- RV1: value 10k -> (none); footprint Potentiometer_THT:Potentiometer_Bourns_3339P_Vertical_HandSoldering -> (none)
- SW1: value Rotary_Encoder_Switch -> (none); footprint Rotary_Encoder:RotaryEncoder_Alps_EC11E-Switch_Vertical_H20mm -> (none)
- U3: value ATMEGA32U4-AU -> (none); footprint Package_QFP:TQFP-44_10x10mm_P0.8mm -> (none)
- U4: value MCP1703A -> (none); footprint Package_TO_SOT_SMD:SOT-23 -> (none)
- U9: value MCP73811T -> (none); footprint Package_TO_SOT_SMD:SOT-23-5 -> (none)
- X1: value MINI-USB-SCHIELD-32005-201 -> (none); footprint Connector_USB:USB_Mini-B_Lumberg_2486_01_Horizontal -> (none)
- Y1: value Crystal -> (none); footprint Crystal:Crystal_SMD_0603-2Pin_6.0x3.5mm_HandSoldering -> (none)
