File: pcb/main/pHMeter.kicad_sch (KiCad schematic)
At the start: 87 parts

Commit message: feat: updated BOM
Parts:
- C11, C20, C21, C23, C6: value (none) -> 10u; footprint (none) -> Capacitor_SMD:C_0805_2012Metric_Pad1.18x1.45mm_HandSolder
- C13, C14: value (none) -> 18p; footprint (none) -> Capacitor_SMD:C_0805_2012Metric_Pad1.15x1.40mm_HandSolder
- C15, C16, C17, C33, C7: value (none) -> 100n; footprint (none) -> Capacitor_SMD:C_0805_2012Metric_Pad1.18x1.45mm_HandSolder
- C18: value (none) -> 1u; footprint (none) -> Capacitor_SMD:C_0805_2012Metric_Pad1.15x1.40mm_HandSolder
- D10, D14, D3, D4, D5: value (none) -> MBR0520LT1G; footprint (none) -> Diode_SMD:D_SOD-123
- D11, D19, D9: value (none) -> YELLOW; footprint (none) -> LED_SMD:LED_0805_2012Metric_Pad1.15x1.40mm_HandSolder
- D12, D13, D17, D18: value (none) -> BLUE; footprint (none) -> LED_SMD:LED_0805_2012Metric_Pad1.15x1.40mm_HandSolder
- D7, D8: value (none) -> GREEN; footprint (none) -> LED_SMD:LED_0805_2012Metric_Pad1.15x1.40mm_HandSolder
- DS1: value (none) -> WC1602A; footprint (none) -> Display:WC1602A
- H1, H2, H3, H4: value (none) -> MountingHole; footprint (none) -> MountingHole:MountingHole_3.2mm_M3
- J1: value (none) -> Conn_02x03_Odd_Even; footprint (none) -> Connector:Tag-Connect_TC2030-IDC-NL_2x03_P1.27mm_Vertical
- J4, J6: value (none) -> AudioJack3_SwitchTR; footprint (none) -> Connector_Audio:Jack_3.5mm_Ledino_KB3SPRS_Horizontal
- J5: value (none) -> RJ12; footprint (none) -> pHMeter:E5566-Q0LK22-L
- J7: value (none) -> SJ; footprint (none) -> Jumper:SolderJumper-2_P1.3mm_Open_RoundedPad1.0x1.5mm
- JP1, JP2: value (none) -> JP1E; footprint (none) -> Connector_PinHeader_2.54mm:PinHeader_1x02_P2.54mm_Vertical
- JP3: value (none) -> acidic; footprint (none) -> Connector_Molex:Molex_KK-254_AE-6410-02A_1x02_P2.54mm_Vertical
- JP4: value (none) -> alkaline; footprint (none) -> Connector_Molex:Molex_KK-254_AE-6410-02A_1x02_P2.54mm_Vertical
- JP5: value (none) -> Bat; footprint (none) -> Connector_Molex:Molex_KK-254_AE-6410-02A_1x02_P2.54mm_Vertical
- JP6: value (none) -> IO3; footprint (none) -> Connector_Molex:Molex_KK-254_AE-6410-02A_1x02_P2.54mm_Vertical
- JP7: value (none) -> IO4; footprint (none) -> Connector_Molex:Molex_KK-254_AE-6410-02A_1x02_P2.54mm_Vertical
- Q1, Q2, Q4, Q5: value (none) -> ZXMS6004; footprint (none) -> Package_TO_SOT_SMD:SOT-23
- Q3: value (none) -> DMP1045; footprint (none) -> Package_TO_SOT_SMD:SOT-23
- R14, R15: value (none) -> 22; footprint (none) -> Resistor_SMD:R_0805_2012Metric_Pad1.15x1.40mm_HandSolder
- R16, R25, R26, R27, R28, R29, R30, R34, R36, R37, R47, R48: value (none) -> 10k; footprint (none) -> Resistor_SMD:R_0805_2012Metric_Pad1.20x1.40mm_HandSolder
- R19, R20, R23, R24, R49, R55: value (none) -> 1k; footprint (none) -> Resistor_SMD:R_0805_2012Metric_Pad1.15x1.40mm_HandSolder
- R21, R51: value (none) -> 4.7k; footprint (none) -> Resistor_SMD:R_0805_2012Metric_Pad1.15x1.40mm_HandSolder
- R22, R32, R33, R53: value (none) -> 100; footprint (none) -> Resistor_SMD:R_0805_2012Metric_Pad1.15x1.40mm_HandSolder
- R31: value (none) -> 0; footprint (none) -> Resistor_SMD:R_0805_2012Metric_Pad1.15x1.40mm_HandSolder
- R35, R38, R45: value (none) -> 1M; footprint (none) -> Resistor_SMD:R_0805_2012Metric_Pad1.15x1.40mm_HandSolder
- R46: value (none) -> 100k; footprint (none) -> Resistor_SMD:R_0805_2012Metric_Pad1.20x1.40mm_HandSolder
- RV1: value (none) -> 10k; footprint (none) -> Potentiometer_THT:Potentiometer_Bourns_3339P_Vertical_HandSoldering
- SW1: value (none) -> Rotary_Encoder_Switch; footprint (none) -> Rotary_Encoder:RotaryEncoder_Alps_EC11E-Switch_Vertical_H20mm
- U3: value (none) -> ATMEGA32U4-AU; footprint (none) -> Package_QFP:TQFP-44_10x10mm_P0.8mm
- U4: value (none) -> MCP1703A; footprint (none) -> Package_TO_SOT_SMD:SOT-23
- U9: value (none) -> MCP73811T; footprint (none) -> Package_TO_SOT_SMD:SOT-23-5
- X1: value (none) -> MINI-USB-SCHIELD-32005-201; footprint (none) -> Connector_USB:USB_Mini-B_Lumberg_2486_01_Horizontal
- Y1: value (none) -> Crystal; footprint (none) -> Crystal:Crystal_SMD_0603-2Pin_6.0x3.5mm_HandSoldering
